File: cad/electronics/AtlasPD/Microcontroller.kicad_pcb (KiCad board)
At the start: 2 copper layers, 24 parts, among them J2 USB_C_Receptacle_USB2.0, SW1 SW_SPST, U2 ATmega328P-AU, U4 CP2104, Y1 CSTNE16M0V53-R0

Commit message: Found a bug, squashed it
Parts:
- added C8: 10uF, Capacitor_SMD:C_0805_2012Metric, F.Cu at (62.6, 67.7)
- added U5: AMS1117-3.3, Package_TO_SOT_SMD:SOT-223-3_TabPin2, F.Cu at (65.7, 73.1)
- moved R4 41.5 mm to (59.1, 59.4), turned to 270 degrees
- moved R12 37.0 mm to (59.1, 62.6), turned to 90 degrees
- moved R5 35.4 mm to (59.1, 65.7), turned to 90 degrees
- moved SW1 30.8 mm to (103.9, 60.3), turned to 180 degrees
- moved R8 28.3 mm to (74.1, 60.7), turned to 180 degrees
- moved C6 26.3 mm to (69.5, 61.8), turned to 270 degrees
- moved U4 25.4 mm to (65.9, 62.8)
- moved R6 24.2 mm to (74.1, 65.5)
- moved D6 24.0 mm to (77.3, 62.3)
- moved J2 22.5 mm to (52.4, 62.8), turned to 270 degrees
- moved R9 22.5 mm to (74.1, 62.3), turned to 180 degrees
- moved Y1 21.7 mm to (93.9, 80.0)
- moved C7 20.4 mm to (60.8, 65.7), turned to 90 degrees
- moved R7 19.2 mm to (74.1, 63.9)
- moved U2 16.1 mm to (98.9, 71.5), turned to 45 degrees
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Routing:
- net (no net): track 0.00 -> 40.6 mm, vias 0 -> 8
- net +5V: track 0.00 -> 20.9 mm, vias 0 -> 6
- net /USB_DP: track 0.00 -> 10.9 mm
- net /USB_DN: track 0.00 -> 7.80 mm
- net Net-(R6-Pad1): track 0.00 -> 6.03 mm
- net GND: track 0.00 -> 5.60 mm, vias 0 -> 9
- net Net-(R7-Pad1): track 0.00 -> 5.59 mm
- net +3V3: track 0.00 -> 5.00 mm
- net Net-(J2-PadA5): track 0.00 -> 3.28 mm
- net Net-(J2-PadB5): track 0.00 -> 2.86 mm
- net Net-(J2-PadB7): track 0.00 -> 2.85 mm
- net Net-(C6-Pad2): track 0.00 -> 1.73 mm
- net Net-(D5-Pad1): track 0.00 -> 1.58 mm
- net Net-(D6-Pad1): track 0.00 -> 1.57 mm
- net Net-(D4-Pad1): track 0.00 -> 1.56 mm
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- added copper zone on F.Cu, net +3V3
- added copper zone on F.Cu, net +5V
- added copper zone on F.Cu, net GND
- added copper zone on F.Cu, net VCC
Other:
- board text added: "3V3"
- board text added: "5V"
