File: cad/electronics/AtlasPD/5V Buck Converter.sch (KiCad schematic (older format))
At the start: 14 parts, among them J1 Conn_01x02_Male, J2 Conn_01x02_Male, U1 LM2678T-ADJ_NOPB

Commit message: Started adding ROS stuff to Arduino, Started Laying out Electrical Diagram
Connections:
- net labels added: +5V
- wire segments 49 -> 51
Changed lines of the file:
@@
 $Descr A4 11693 8268
 encoding utf-8
-Sheet 2 3
+Sheet 2 4
 Title "Atlas Power Distribution Board"
 Date ""
@@
 Connection ~ 7250 1700
 Wire Wire Line
-	7800 1700 8500 1700
+	7800 1700 8400 1700
 Connection ~ 7800 1700
 Wire Wire Line
@@
 Text Notes 2750 1200 2    118  ~ 24
 5V Buck Converter
+$Comp
+L power:+5V #PWR?
+U 1 1 61270FB8
+P 8400 1500
+F 0 "#PWR?" H 8400 1350 50  0001 C CNN
+F 1 "+5V" H 8415 1673 50  0000 C CNN
+F 2 "" H 8400 1500 50  0001 C CNN
+F 3 "" H 8400 1500 50  0001 C CNN
+	1    8400 1500
+	1    0    0    -1
+$EndComp
+Wire Wire Line
+	8400 1500 8400 1700
+Connection ~ 8400 1700
+Wire Wire Line
+	8400 1700 8500 1700
 $EndSCHEMATC

Commit message: Added LDO
Connections:
- net labels added: Output
- net labels removed: +5V
- wire segments 51 -> 52
Changed lines of the file:
@@
 Text Notes 2750 1200 2    118  ~ 24
 5V Buck Converter
-$Comp
-L power:+5V #PWR?
-U 1 1 61270FB8
-P 8400 1500
-F 0 "#PWR?" H 8400 1350 50  0001 C CNN
-F 1 "+5V" H 8415 1673 50  0000 C CNN
-F 2 "" H 8400 1500 50  0001 C CNN
-F 3 "" H 8400 1500 50  0001 C CNN
-	1    8400 1500
-	1    0    0    -1
-$EndComp
 Wire Wire Line
 	8400 1500 8400 1700
@@
 Wire Wire Line
 	8400 1700 8500 1700
+Text HLabel 8600 1500 2    50   Input ~ 0
+Output
+Wire Wire Line
+	8600 1500 8400 1500
 $EndSCHEMATC

Commit message: PCB Changes to 5V Regulator
Parts:
- L1: footprint Inductor_THT:L_Axial_L6.6mm_D2.7mm_P10.16mm_Horizontal_Vishay_IM-2 -> Inductor_SMD:L_TDK_NLV32_3.2x2.5mm
Connections:
- no-connect marks 0 -> 1
Changed lines of the file:
@@
 F 0 "L1" V 5490 1700 50  0000 C CNN
 F 1 "22 uH" V 5399 1700 50  0000 C CNN
-F 2 "Inductor_THT:L_Axial_L6.6mm_D2.7mm_P10.16mm_Horizontal_Vishay_IM-2" H 5300 1700 50  0001 C CNN
+F 2 "Inductor_SMD:L_TDK_NLV32_3.2x2.5mm" H 5300 1700 50  0001 C CNN
 F 3 "~" H 5300 1700 50  0001 C CNN
 	1    5300 1700
@@
 Wire Wire Line
 	8600 1500 8400 1500
+NoConn ~ 3300 1800
 $EndSCHEMATC

Commit message: More PCB changes
Parts:
- D1: footprint Capacitor_SMD:C_0805_2012Metric -> Diode_SMD:D_SOD-128
Changed lines of the file:
@@
 F 0 "D1" V 5004 2230 50  0000 L CNN
 F 1 "D_Schottky" V 5095 2230 50  0000 L CNN
-F 2 "Capacitor_SMD:C_0805_2012Metric" H 5050 2150 50  0001 C CNN
+F 2 "Diode_SMD:D_SOD-128" H 5050 2150 50  0001 C CNN
 F 3 "~" H 5050 2150 50  0001 C CNN
 	1    5050 2150

Commit message: More Electronics design work
Parts:
- removed J2: Conn_01x02_Male, Connector_PinHeader_2.54mm:PinHeader_1x02_P2.54mm_Vertical, symbol Connector:Conn_01x02_Male
- added C8: 10uF, Capacitor_SMD:C_0805_2012Metric, symbol Device:C
- added U5: AMS1117-3.3, Package_TO_SOT_SMD:SOT-223-3_TabPin2, symbol Regulator_Linear:AMS1117-3.3
- C5: footprint Capacitor_THT:CP_Radial_D5.0mm_P2.50mm -> Capacitor_THT:CP_Radial_D10.0mm_P3.50mm
Connections:
- net labels added: +3.3V, +5V
- net labels removed: Output
Other:
- note added: "3.3V LDO"
Changed lines of the file:
@@
 $Descr A4 11693 8268
 encoding utf-8
-Sheet 2 4
+Sheet 4 4
 Title "Atlas Power Distribution Board"
 Date ""
@@
 F 0 "C5" H 6415 2196 50  0000 L CNN
 F 1 "1000uF" H 6415 2105 50  0000 L CNN
-F 2 "Capacitor_THT:CP_Radial_D5.0mm_P2.50mm" H 6300 2150 50  0001 C CNN
+F 2 "Capacitor_THT:CP_Radial_D10.0mm_P3.50mm" H 6300 2150 50  0001 C CNN
 F 3 "~" H 6300 2150 50  0001 C CNN
 	1    6300 2150
@@
 	5050 1200 5050 1700
 $Comp
-L Connector:Conn_01x02_Male J2
-U 1 1 60A2CCDC
-P 8700 1800
-F 0 "J2" H 8672 1682 50  0000 R CNN
-F 1 "Conn_01x02_Male" H 8672 1773 50  0000 R CNN
-F 2 "Connector_PinHeader_2.54mm:PinHeader_1x02_P2.54mm_Vertical" H 8700 1800 50  0001 C CNN
-F 3 "~" H 8700 1800 50  0001 C CNN
-	1    8700 1800
-	-1   0    0    1
-$EndComp
-Wire Wire Line
-	8500 1800 8500 2650
-$Comp
 L Device:R R3
 U 1 1 60A2CCE3
@@
 Connection ~ 7250 1700
 Wire Wire Line
-	7800 1700 8400 1700
-Connection ~ 7800 1700
-Wire Wire Line
 	7800 2100 7800 2250
 Wire Wire Line
 	7800 2550 7800 2650
 Wire Wire Line
-	7800 2650 8500 2650
-Wire Wire Line
 	7800 2650 7250 2650
-Connection ~ 7800 2650
 Connection ~ 7250 2650
 Text Notes 2750 1200 2    118  ~ 24
 5V Buck Converter
-Wire Wire Line
-	8400 1500 8400 1700
-Connection ~ 8400 1700
-Wire Wire Line
-	8400 1700 8500 1700
-Text HLabel 8600 1500 2    50   Input ~ 0
-Output
-Wire Wire Line
-	8600 1500 8400 1500
 NoConn ~ 3300 1800
+$Comp
+L power:+5V #PWR0102
+U 1 1 615F3821
+P 7800 1600
+F 0 "#PWR0102" H 7800 1450 50  0001 C CNN
+F 1 "+5V" H 7815 1773 50  0000 C CNN
+F 2 "" H 7800 1600 50  0001 C CNN
+F 3 "" H 7800 1600 50  0001 C CNN
+	1    7800 1600
+	1    0    0    -1
+$EndComp
+Wire Wire Line
+	7800 1600 7800 1700
+Connection ~ 7800 1700
+$Comp
+L Regulator_Linear:AMS1117-3.3 U5
+U 1 1 616268E3
+P 2150 4200
+F 0 "U5" H 2150 4442 50  0000 C CNN
+F 1 "AMS1117-3.3" H 2150 4351 50  0000 C CNN
+F 2 "Package_TO_SOT_SMD:SOT-223-3_TabPin2" H 2150 4400 50  0001 C CNN
+F 3 "http://www.advanced-monolithic.com/pdf/ds1117.pdf" H 2250 3950 50  0001 C CNN
+	1    2150 4200
+	1    0    0    -1
+$EndComp
+Text Notes 1350 3450 0    118  ~ 24
+3.3V LDO
+$Comp
+L power:+5V #PWR015
+U 1 1 6162A464
+P 1700 3800
+F 0 "#PWR015" H 1700 3650 50  0001 C CNN
+F 1 "+5V" H 1715 3973 50  0000 C CNN
+F 2 "" H 1700 3800 50  0001 C CNN
+F 3 "" H 1700 3800 50  0001 C CNN
+	1    1700 3800
+	1    0    0    -1
+$EndComp
+$Comp
+L power:+3.3V #PWR017
+U 1 1 6162B28C
+P 2550 3800
+F 0 "#PWR017" H 2550 3650 50  0001 C CNN
+F 1 "+3.3V" H 2565 3973 50  0000 C CNN
+F 2 "" H 2550 3800 50  0001 C CNN
+F 3 "" H 2550 3800 50  0001 C CNN
+	1    2550 3800
+	1    0    0    -1
+$EndComp
+$Comp
+L power:GND #PWR016
+U 1 1 6162B9AF
+P 2150 4550
+F 0 "#PWR016" H 2150 4300 50  0001 C CNN
+F 1 "GND" H 2155 4377 50  0000 C CNN
+F 2 "" H 2150 4550 50  0001 C CNN
+F 3 "" H 2150 4550 50  0001 C CNN
+	1    2150 4550
+	1    0    0    -1
+$EndComp
+Wire Wire Line
+	1700 4200 1850 4200
+Wire Wire Line
+	2450 4200 2550 4200
+Wire Wire Line
+	2550 4200 2550 4100
+Wire Wire Line
+	2150 4500 2150 4550
+$Comp
+L Device:C C8
+U 1 1 6163B27F
+P 2550 3950
+F 0 "C8" H 2665 3996 50  0000 L CNN
+F 1 "10uF" H 2665 3905 50  0000 L CNN
+F 2 "Capacitor_SMD:C_0805_2012Metric" H 2588 3800 50  0001 C CNN
+F 3 "~" H 2550 3950 50  0001 C CNN
+	1    2550 3950
+	1    0    0    -1
+$EndComp
+Wire Wire Line
+	1700 3800 1700 4200
 $EndSCHEMATC

Commit message: Project Restructuring for ease of design and other stuff
Parts:
- removed J1: Conn_01x02_Male, Connector_PinHeader_2.54mm:PinHeader_1x02_P2.54mm_Vertical, symbol Connector:Conn_01x02_Male
- added BT1, BT2: Battery_Cell, Battery:BatteryHolder_Keystone_1042_1x18650, symbol Device:Battery_Cell
Connections:
- net labels added: +BATT
- wire segments 52 -> 55
Changed lines of the file:
@@
 encoding utf-8
 Sheet 4 4
-Title "Atlas Power Distribution Board"
-Date ""
-Rev "0.1"
+Title "Atlas Power Board"
+Date "2021-10-08"
+Rev "0.2"
 Comp ""
 Comment1 "Manpreet Singh"
@@
 $EndComp
 $Comp
-L Connector:Conn_01x02_Male J1
-U 1 1 60A2CC8E
-P 1450 1700
-F 0 "J1" H 1558 1881 50  0000 C CNN
-F 1 "Conn_01x02_Male" H 1558 1790 50  0000 C CNN
-F 2 "Connector_PinHeader_2.54mm:PinHeader_1x02_P2.54mm_Vertical" H 1450 1700 50  0001 C CNN
-F 3 "~" H 1450 1700 50  0001 C CNN
-	1    1450 1700
-	1    0    0    -1
-$EndComp
-$Comp
 L Device:L L1
 U 1 1 60A2CC94
@@
 	0    -1   -1   0
 $EndComp
-Wire Wire Line
-	1650 1700 2050 1700
 $Comp
 L power:GND #PWR0101
@@
 $EndComp
 Wire Wire Line
-	1650 1800 1650 2650
-Wire Wire Line
 	2050 1950 2050 1700
 Connection ~ 2050 1700
@@
 Wire Wire Line
 	2050 2650 1650 2650
-Connection ~ 1650 2650
 Wire Wire Line
 	1650 2650 1650 2700
@@
 Wire Wire Line
 	1700 3800 1700 4200
+$Comp
+L Device:Battery_Cell BT1
+U 1 1 61621A89
+P 1050 2050
+F 0 "BT1" H 1168 2146 50  0000 L CNN
+F 1 "Battery_Cell" H 1168 2055 50  0000 L CNN
+F 2 "Battery:BatteryHolder_Keystone_1042_1x18650" V 1050 2110 50  0001 C CNN
+F 3 "~" V 1050 2110 50  0001 C CNN
+	1    1050 2050
+	1    0    0    -1
+$EndComp
+$Comp
+L Device:Battery_Cell BT2
+U 1 1 616223C5
+P 1050 2350
+F 0 "BT2" H 1168 2446 50  0000 L CNN
+F 1 "Battery_Cell" H 1168 2355 50  0000 L CNN
+F 2 "Battery:BatteryHolder_Keystone_1042_1x18650" V 1050 2410 50  0001 C CNN
+F 3 "~" V 1050 2410 50  0001 C CNN
+	1    1050 2350
+	1    0    0    -1
+$EndComp
+Wire Wire Line
+	1050 1850 1050 1700
+Wire Wire Line
+	1050 1700 2050 1700
+Wire Wire Line
+	1050 2450 1050 2650
+Wire Wire Line
+	1050 2650 1650 2650
+Connection ~ 1650 2650
+$Comp
+L power:+BATT #PWR?
+U 1 1 616386ED
+P 1050 1550
+F 0 "#PWR?" H 1050 1400 50  0001 C CNN
+F 1 "+BATT" H 1065 1723 50  0000 C CNN
+F 2 "" H 1050 1550 50  0001 C CNN
+F 3 "" H 1050 1550 50  0001 C CNN
+	1    1050 1550
+	1    0    0    -1
+$EndComp
+Wire Wire Line
+	1050 1550 1050 1700
+Connection ~ 1050 1700
 $EndSCHEMATC

Commit message: Found a bug, squashed it
Parts:
- C8: footprint Capacitor_SMD:C_0805_2012Metric -> Capacitor_SMD:C_0603_1608Metric
Connections:
- wire segments 55 -> 56
Other:
- moved on the sheet: C8
Changed lines of the file:
@@
 	2450 4200 2550 4200
-Wire Wire Line
-	2550 4200 2550 4100
 Wire Wire Line
 	2150 4500 2150 4550
@@
 L Device:C C8
 U 1 1 6163B27F
-P 2550 3950
-F 0 "C8" H 2665 3996 50  0000 L CNN
-F 1 "10uF" H 2665 3905 50  0000 L CNN
-F 2 "Capacitor_SMD:C_0805_2012Metric" H 2588 3800 50  0001 C CNN
-F 3 "~" H 2550 3950 50  0001 C CNN
-	1    2550 3950
+P 2550 4350
+F 0 "C8" H 2665 4396 50  0000 L CNN
+F 1 "10uF" H 2665 4305 50  0000 L CNN
+F 2 "Capacitor_SMD:C_0603_1608Metric" H 2588 4200 50  0001 C CNN
+F 3 "~" H 2550 4350 50  0001 C CNN
+	1    2550 4350
 	1    0    0    -1
 $EndComp
@@
 Connection ~ 1650 2650
 $Comp
-L power:+BATT #PWR?
+L power:+BATT #PWR0109
 U 1 1 616386ED
 P 1050 1550
-F 0 "#PWR?" H 1050 1400 50  0001 C CNN
+F 0 "#PWR0109" H 1050 1400 50  0001 C CNN
 F 1 "+BATT" H 1065 1723 50  0000 C CNN
 F 2 "" H 1050 1550 50  0001 C CNN
@@
 	1050 1550 1050 1700
 Connection ~ 1050 1700
+Connection ~ 2550 4200
+Wire Wire Line
+	2550 3800 2550 4200
+Wire Wire Line
+	2550 4500 2150 4500
+Connection ~ 2150 4500
 $EndSCHEMATC

Commit message: Power board layout
Parts:
- U1: footprint LM2678:TO127P1041X469X2199-7N -> SamacSys_Parts:TO127P1435X464-8N
Changed lines of the file:
@@
 $Descr A4 11693 8268
 encoding utf-8
-Sheet 4 4
+Sheet 1 1
 Title "Atlas Power Board"
 Date "2021-10-08"
@@
 F 0 "U1" H 4000 2367 50  0000 C CNN
 F 1 "LM2678T-ADJ_NOPB" H 4000 2276 50  0000 C CNN
-F 2 "LM2678:TO127P1041X469X2199-7N" H 4000 1900 50  0001 L BNN
+F 2 "SamacSys_Parts:TO127P1435X464-8N" H 4000 1900 50  0001 L BNN
 F 3 "" H 4000 1900 50  0001 L BNN
 F 4 "TEXAS INSTRUMENTS" H 4000 1900 50  0001 L BNN "MANUFACTURER"
@@
 	1    0    0    -1
 $EndComp
-Text Notes 1350 3450 0    118  ~ 24
+Text Notes 1100 3450 0    118  ~ 24
 3.3V LDO
 $Comp
