File: cad/electronics/AtlasPD/5V Buck Converter.sch (KiCad schematic (older format))
At the start: 16 parts, among them U1 LM2678T-ADJ_NOPB, U5 AMS1117-3.3

Commit message: First Board Layout done
Parts:
- added J5: Conn_01x04, Connector_JST:JST_PH_B4B-PH-K_1x04_P2.00mm_Vertical, symbol Connector_Generic:Conn_01x04
- renumbered C4 to C10, C5 to C11, C1 to C6, C2 to C7, C3 to C9, D1 to D5, D2 to D6, R1 to R10, R2 to R11, R3 to R12, U5 to U6, U1 to U7
Other:
- note added: "Power Output Connector"
Changed lines of the file:
@@
 $Descr A4 11693 8268
 encoding utf-8
-Sheet 1 1
+Sheet 4 4
 Title "Atlas Power Board"
 Date "2021-10-08"
@@
 $EndDescr
 $Comp
-L LM2678T-ADJ/NOPB:LM2678T-ADJ_NOPB U1
+L LM2678T-ADJ/NOPB:LM2678T-ADJ_NOPB U7
 U 1 1 60A2CC5E
 P 4000 1900
-F 0 "U1" H 4000 2367 50  0000 C CNN
+F 0 "U7" H 4000 2367 50  0000 C CNN
 F 1 "LM2678T-ADJ_NOPB" H 4000 2276 50  0000 C CNN
 F 2 "SamacSys_Parts:TO127P1435X464-8N" H 4000 1900 50  0001 L BNN
@@
 $EndComp
 $Comp
-L Device:C C2
+L Device:C C7
 U 1 1 60A2CC64
 P 2450 2100
-F 0 "C2" H 2565 2146 50  0000 L CNN
+F 0 "C7" H 2565 2146 50  0000 L CNN
 F 1 "10uF" H 2565 2055 50  0000 L CNN
 F 2 "Capacitor_SMD:C_0805_2012Metric" H 2488 1950 50  0001 C CNN
@@
 $EndComp
 $Comp
-L Device:C C4
+L Device:C C10
 U 1 1 60A2CC6A
 P 5950 2150
-F 0 "C4" H 6065 2196 50  0000 L CNN
+F 0 "C10" H 6065 2196 50  0000 L CNN
 F 1 "10uF" H 6065 2105 50  0000 L CNN
 F 2 "Capacitor_SMD:C_0805_2012Metric" H 5988 2000 50  0001 C CNN
@@
 $EndComp
 $Comp
-L Device:CP1 C1
+L Device:CP1 C6
 U 1 1 60A2CC70
 P 2050 2100
-F 0 "C1" H 2165 2146 50  0000 L CNN
+F 0 "C6" H 2165 2146 50  0000 L CNN
 F 1 "220uF" H 2165 2055 50  0000 L CNN
 F 2 "Capacitor_THT:CP_Radial_D5.0mm_P2.50mm" H 2050 2100 50  0001 C CNN
@@
 $EndComp
 $Comp
-L Device:CP1 C5
+L Device:CP1 C11
 U 1 1 60A2CC76
 P 6300 2150
-F 0 "C5" H 6415 2196 50  0000 L CNN
+F 0 "C11" H 6415 2196 50  0000 L CNN
 F 1 "1000uF" H 6415 2105 50  0000 L CNN
 F 2 "Capacitor_THT:CP_Radial_D10.0mm_P3.50mm" H 6300 2150 50  0001 C CNN
@@
 $EndComp
 $Comp
-L Device:D_Schottky D1
+L Device:D_Schottky D5
 U 1 1 60A2CC7C
 P 5050 2150
-F 0 "D1" V 5004 2230 50  0000 L CNN
+F 0 "D5" V 5004 2230 50  0000 L CNN
 F 1 "D_Schottky" V 5095 2230 50  0000 L CNN
 F 2 "Diode_SMD:D_SOD-128" H 5050 2150 50  0001 C CNN
@@
 $EndComp
 $Comp
-L Device:R R1
+L Device:R R10
 U 1 1 60A2CC82
 P 7250 1950
-F 0 "R1" H 7320 1996 50  0000 L CNN
+F 0 "R10" H 7320 1996 50  0000 L CNN
 F 1 "3.16k" H 7320 1905 50  0000 L CNN
 F 2 "Resistor_SMD:R_0805_2012Metric" V 7180 1950 50  0001 C CNN
@@
 $EndComp
 $Comp
-L Device:R R2
+L Device:R R11
 U 1 1 60A2CC88
 P 7250 2400
-F 0 "R2" H 7320 2446 50  0000 L CNN
+F 0 "R11" H 7320 2446 50  0000 L CNN
 F 1 "1k" H 7320 2355 50  0000 L CNN
 F 2 "Resistor_SMD:R_0805_2012Metric" V 7180 2400 50  0001 C CNN
@@
 $EndComp
 $Comp
-L power:GND #PWR0101
+L power:GND #PWR034
 U 1 1 60A2CC9B
 P 1650 2700
-F 0 "#PWR0101" H 1650 2450 50  0001 C CNN
+F 0 "#PWR034" H 1650 2450 50  0001 C CNN
 F 1 "GND" H 1655 2527 50  0000 C CNN
 F 2 "" H 1650 2700 50  0001 C CNN
@@
 Connection ~ 6300 2650
 $Comp
-L Device:C C3
+L Device:C C9
 U 1 1 60A2CCCA
 P 3850 1200
-F 0 "C3" V 3598 1200 50  0000 C CNN
+F 0 "C9" V 3598 1200 50  0000 C CNN
 F 1 "10uF" V 3689 1200 50  0000 C CNN
 F 2 "Capacitor_SMD:C_0805_2012Metric" H 3888 1050 50  0001 C CNN
@@
 	5050 1200 5050 1700
 $Comp
-L Device:R R3
+L Device:R R12
 U 1 1 60A2CCE3
 P 7800 2400
-F 0 "R3" H 7870 2446 50  0000 L CNN
+F 0 "R12" H 7870 2446 50  0000 L CNN
 F 1 "1k" H 7870 2355 50  0000 L CNN
 F 2 "Resistor_SMD:R_0805_2012Metric" V 7730 2400 50  0001 C CNN
@@
 $EndComp
 $Comp
-L Device:LED D2
+L Device:LED D6
 U 1 1 60A2CCE9
 P 7800 1950
-F 0 "D2" V 7839 1832 50  0000 R CNN
+F 0 "D6" V 7839 1832 50  0000 R CNN
 F 1 "LED" V 7748 1832 50  0000 R CNN
 F 2 "LED_SMD:LED_0805_2012Metric" H 7800 1950 50  0001 C CNN
@@
 NoConn ~ 3300 1800
 $Comp
-L power:+5V #PWR0102
+L power:+5V #PWR042
 U 1 1 615F3821
 P 7800 1600
-F 0 "#PWR0102" H 7800 1450 50  0001 C CNN
+F 0 "#PWR042" H 7800 1450 50  0001 C CNN
 F 1 "+5V" H 7815 1773 50  0000 C CNN
 F 2 "" H 7800 1600 50  0001 C CNN
@@
 Connection ~ 7800 1700
 $Comp
-L Regulator_Linear:AMS1117-3.3 U5
+L Regulator_Linear:AMS1117-3.3 U6
 U 1 1 616268E3
 P 2150 4200
-F 0 "U5" H 2150 4442 50  0000 C CNN
+F 0 "U6" H 2150 4442 50  0000 C CNN
 F 1 "AMS1117-3.3" H 2150 4351 50  0000 C CNN
 F 2 "Package_TO_SOT_SMD:SOT-223-3_TabPin2" H 2150 4400 50  0001 C CNN
@@
 3.3V LDO
 $Comp
-L power:+5V #PWR015
+L power:+5V #PWR035
 U 1 1 6162A464
 P 1700 3800
-F 0 "#PWR015" H 1700 3650 50  0001 C CNN
+F 0 "#PWR035" H 1700 3650 50  0001 C CNN
 F 1 "+5V" H 1715 3973 50  0000 C CNN
 F 2 "" H 1700 3800 50  0001 C CNN
@@
 $EndComp
 $Comp
-L power:+3.3V #PWR017
+L power:+3.3V #PWR037
 U 1 1 6162B28C
 P 2550 3800
-F 0 "#PWR017" H 2550 3650 50  0001 C CNN
+F 0 "#PWR037" H 2550 3650 50  0001 C CNN
 F 1 "+3.3V" H 2565 3973 50  0000 C CNN
 F 2 "" H 2550 3800 50  0001 C CNN
@@
 $EndComp
 $Comp
-L power:GND #PWR016
+L power:GND #PWR036
 U 1 1 6162B9AF
 P 2150 4550
-F 0 "#PWR016" H 2150 4300 50  0001 C CNN
+F 0 "#PWR036" H 2150 4300 50  0001 C CNN
 F 1 "GND" H 2155 4377 50  0000 C CNN
 F 2 "" H 2150 4550 50  0001 C CNN
@@
 Connection ~ 1650 2650
 $Comp
-L power:+BATT #PWR0109
+L power:+BATT #PWR033
 U 1 1 616386ED
 P 1050 1550
-F 0 "#PWR0109" H 1050 1400 50  0001 C CNN
+F 0 "#PWR033" H 1050 1400 50  0001 C CNN
 F 1 "+BATT" H 1065 1723 50  0000 C CNN
 F 2 "" H 1050 1550 50  0001 C CNN
@@
 	2550 4500 2150 4500
 Connection ~ 2150 4500
+$Comp
+L power:+5V #PWR040
+U 1 1 6168DE84
+P 4450 4000
+F 0 "#PWR040" H 4450 3850 50  0001 C CNN
+F 1 "+5V" V 4450 4200 50  0000 C CNN
+F 2 "" H 4450 4000 50  0001 C CNN
+F 3 "" H 4450 4000 50  0001 C CNN
+	1    4450 4000
+	0    -1   -1   0
+$EndComp
+$Comp
+L power:GND #PWR039
+U 1 1 6168E347
+P 4450 4100
+F 0 "#PWR039" H 4450 3850 50  0001 C CNN
+F 1 "GND" V 4450 3900 50  0000 C CNN
+F 2 "" H 4450 4100 50  0001 C CNN
+F 3 "" H 4450 4100 50  0001 C CNN
+	1    4450 4100
+	0    1    1    0
+$EndComp
+$Comp
+L Connector_Generic:Conn_01x04 J5
+U 1 1 616A0CC6
+P 4650 4100
+F 0 "J5" H 4730 4092 50  0000 L CNN
+F 1 "Conn_01x04" H 4730 4001 50  0000 L CNN
+F 2 "Connector_JST:JST_PH_B4B-PH-K_1x04_P2.00mm_Vertical" H 4650 4100 50  0001 C CNN
+F 3 "~" H 4650 4100 50  0001 C CNN
+	1    4650 4100
+	1    0    0    -1
+$EndComp
+$Comp
+L power:+BATT #PWR0103
+U 1 1 616AC55C
+P 4450 4200
+F 0 "#PWR0103" H 4450 4050 50  0001 C CNN
+F 1 "+BATT" V 4450 4450 50  0000 C CNN
+F 2 "" H 4450 4200 50  0001 C CNN
+F 3 "" H 4450 4200 50  0001 C CNN
+	1    4450 4200
+	0    -1   -1   0
+$EndComp
+$Comp
+L power:GND #PWR0104
+U 1 1 616AD750
+P 4450 4300
+F 0 "#PWR0104" H 4450 4050 50  0001 C CNN
+F 1 "GND" V 4450 4100 50  0000 C CNN
+F 2 "" H 4450 4300 50  0001 C CNN
+F 3 "" H 4450 4300 50  0001 C CNN
+	1    4450 4300
+	0    1    1    0
+$EndComp
+Text Notes 3900 3450 0    118  ~ 24
+Power Output Connector
 $EndSCHEMATC

Commit message: Layout updates
Parts:
- renumbered BT1 to BT401, BT2 to BT402, C6 to C401, C7 to C402, C8 to C403, C9 to C404, C10 to C405, C11 to C406, D5 to D401, D6 to D402, J5 to J401, L1 to L401, R10 to R401, R11 to R402, R12 to R403, U6 to U401, U7 to U402
Changed lines of the file:
@@
 $EndDescr
 $Comp
-L LM2678T-ADJ/NOPB:LM2678T-ADJ_NOPB U7
+L LM2678T-ADJ/NOPB:LM2678T-ADJ_NOPB U402
 U 1 1 60A2CC5E
 P 4000 1900
-F 0 "U7" H 4000 2367 50  0000 C CNN
+F 0 "U402" H 4000 2367 50  0000 C CNN
 F 1 "LM2678T-ADJ_NOPB" H 4000 2276 50  0000 C CNN
 F 2 "SamacSys_Parts:TO127P1435X464-8N" H 4000 1900 50  0001 L BNN
@@
 $EndComp
 $Comp
-L Device:C C7
+L Device:C C402
 U 1 1 60A2CC64
 P 2450 2100
-F 0 "C7" H 2565 2146 50  0000 L CNN
+F 0 "C402" H 2565 2146 50  0000 L CNN
 F 1 "10uF" H 2565 2055 50  0000 L CNN
 F 2 "Capacitor_SMD:C_0805_2012Metric" H 2488 1950 50  0001 C CNN
@@
 $EndComp
 $Comp
-L Device:C C10
+L Device:C C405
 U 1 1 60A2CC6A
 P 5950 2150
-F 0 "C10" H 6065 2196 50  0000 L CNN
+F 0 "C405" H 6065 2196 50  0000 L CNN
 F 1 "10uF" H 6065 2105 50  0000 L CNN
 F 2 "Capacitor_SMD:C_0805_2012Metric" H 5988 2000 50  0001 C CNN
@@
 $EndComp
 $Comp
-L Device:CP1 C6
+L Device:CP1 C401
 U 1 1 60A2CC70
 P 2050 2100
-F 0 "C6" H 2165 2146 50  0000 L CNN
+F 0 "C401" H 2165 2146 50  0000 L CNN
 F 1 "220uF" H 2165 2055 50  0000 L CNN
 F 2 "Capacitor_THT:CP_Radial_D5.0mm_P2.50mm" H 2050 2100 50  0001 C CNN
@@
 $EndComp
 $Comp
-L Device:CP1 C11
+L Device:CP1 C406
 U 1 1 60A2CC76
 P 6300 2150
-F 0 "C11" H 6415 2196 50  0000 L CNN
+F 0 "C406" H 6415 2196 50  0000 L CNN
 F 1 "1000uF" H 6415 2105 50  0000 L CNN
 F 2 "Capacitor_THT:CP_Radial_D10.0mm_P3.50mm" H 6300 2150 50  0001 C CNN
@@
 $EndComp
 $Comp
-L Device:D_Schottky D5
+L Device:D_Schottky D401
 U 1 1 60A2CC7C
 P 5050 2150
-F 0 "D5" V 5004 2230 50  0000 L CNN
+F 0 "D401" V 5004 2230 50  0000 L CNN
 F 1 "D_Schottky" V 5095 2230 50  0000 L CNN
 F 2 "Diode_SMD:D_SOD-128" H 5050 2150 50  0001 C CNN
@@
 $EndComp
 $Comp
-L Device:R R10
+L Device:R R401
 U 1 1 60A2CC82
 P 7250 1950
-F 0 "R10" H 7320 1996 50  0000 L CNN
+F 0 "R401" H 7320 1996 50  0000 L CNN
 F 1 "3.16k" H 7320 1905 50  0000 L CNN
 F 2 "Resistor_SMD:R_0805_2012Metric" V 7180 1950 50  0001 C CNN
@@
 $EndComp
 $Comp
-L Device:R R11
+L Device:R R402
 U 1 1 60A2CC88
 P 7250 2400
-F 0 "R11" H 7320 2446 50  0000 L CNN
+F 0 "R402" H 7320 2446 50  0000 L CNN
 F 1 "1k" H 7320 2355 50  0000 L CNN
 F 2 "Resistor_SMD:R_0805_2012Metric" V 7180 2400 50  0001 C CNN
@@
 $EndComp
 $Comp
-L Device:L L1
+L Device:L L401
 U 1 1 60A2CC94
 P 5300 1700
-F 0 "L1" V 5490 1700 50  0000 C CNN
+F 0 "L401" V 5490 1700 50  0000 C CNN
 F 1 "22 uH" V 5399 1700 50  0000 C CNN
 F 2 "Inductor_SMD:L_TDK_NLV32_3.2x2.5mm" H 5300 1700 50  0001 C CNN
@@
 $EndComp
 $Comp
-L power:GND #PWR034
+L power:GND #PWR0402
 U 1 1 60A2CC9B
 P 1650 2700
-F 0 "#PWR034" H 1650 2450 50  0001 C CNN
+F 0 "#PWR0402" H 1650 2450 50  0001 C CNN
 F 1 "GND" H 1655 2527 50  0000 C CNN
 F 2 "" H 1650 2700 50  0001 C CNN
@@
 Connection ~ 6300 2650
 $Comp
-L Device:C C9
+L Device:C C404
 U 1 1 60A2CCCA
 P 3850 1200
-F 0 "C9" V 3598 1200 50  0000 C CNN
+F 0 "C404" V 3598 1200 50  0000 C CNN
 F 1 "10uF" V 3689 1200 50  0000 C CNN
 F 2 "Capacitor_SMD:C_0805_2012Metric" H 3888 1050 50  0001 C CNN
@@
 	5050 1200 5050 1700
 $Comp
-L Device:R R12
+L Device:R R403
 U 1 1 60A2CCE3
 P 7800 2400
-F 0 "R12" H 7870 2446 50  0000 L CNN
+F 0 "R403" H 7870 2446 50  0000 L CNN
 F 1 "1k" H 7870 2355 50  0000 L CNN
 F 2 "Resistor_SMD:R_0805_2012Metric" V 7730 2400 50  0001 C CNN
@@
 $EndComp
 $Comp
-L Device:LED D6
+L Device:LED D402
 U 1 1 60A2CCE9
 P 7800 1950
-F 0 "D6" V 7839 1832 50  0000 R CNN
+F 0 "D402" V 7839 1832 50  0000 R CNN
 F 1 "LED" V 7748 1832 50  0000 R CNN
 F 2 "LED_SMD:LED_0805_2012Metric" H 7800 1950 50  0001 C CNN
@@
 NoConn ~ 3300 1800
 $Comp
-L power:+5V #PWR042
+L power:+5V #PWR0410
 U 1 1 615F3821
 P 7800 1600
-F 0 "#PWR042" H 7800 1450 50  0001 C CNN
+F 0 "#PWR0410" H 7800 1450 50  0001 C CNN
 F 1 "+5V" H 7815 1773 50  0000 C CNN
 F 2 "" H 7800 1600 50  0001 C CNN
@@
 Connection ~ 7800 1700
 $Comp
-L Regulator_Linear:AMS1117-3.3 U6
+L Regulator_Linear:AMS1117-3.3 U401
 U 1 1 616268E3
 P 2150 4200
-F 0 "U6" H 2150 4442 50  0000 C CNN
+F 0 "U401" H 2150 4442 50  0000 C CNN
 F 1 "AMS1117-3.3" H 2150 4351 50  0000 C CNN
 F 2 "Package_TO_SOT_SMD:SOT-223-3_TabPin2" H 2150 4400 50  0001 C CNN
@@
 3.3V LDO
 $Comp
-L power:+5V #PWR035
+L power:+5V #PWR0403
 U 1 1 6162A464
 P 1700 3800
-F 0 "#PWR035" H 1700 3650 50  0001 C CNN
+F 0 "#PWR0403" H 1700 3650 50  0001 C CNN
 F 1 "+5V" H 1715 3973 50  0000 C CNN
 F 2 "" H 1700 3800 50  0001 C CNN
@@
 $EndComp
 $Comp
-L power:+3.3V #PWR037
+L power:+3.3V #PWR0405
 U 1 1 6162B28C
 P 2550 3800
-F 0 "#PWR037" H 2550 3650 50  0001 C CNN
+F 0 "#PWR0405" H 2550 3650 50  0001 C CNN
 F 1 "+3.3V" H 2565 3973 50  0000 C CNN
 F 2 "" H 2550 3800 50  0001 C CNN
@@
 $EndComp
 $Comp
-L power:GND #PWR036
+L power:GND #PWR0404
 U 1 1 6162B9AF
 P 2150 4550
-F 0 "#PWR036" H 2150 4300 50  0001 C CNN
+F 0 "#PWR0404" H 2150 4300 50  0001 C CNN
 F 1 "GND" H 2155 4377 50  0000 C CNN
 F 2 "" H 2150 4550 50  0001 C CNN
@@
 	2150 4500 2150 4550
 $Comp
-L Device:C C8
+L Device:C C403
 U 1 1 6163B27F
 P 2550 4350
-F 0 "C8" H 2665 4396 50  0000 L CNN
+F 0 "C403" H 2665 4396 50  0000 L CNN
 F 1 "10uF" H 2665 4305 50  0000 L CNN
 F 2 "Capacitor_SMD:C_0603_1608Metric" H 2588 4200 50  0001 C CNN
@@
 	1700 3800 1700 4200
 $Comp
-L Device:Battery_Cell BT1
+L Device:Battery_Cell BT401
 U 1 1 61621A89
 P 1050 2050
-F 0 "BT1" H 1168 2146 50  0000 L CNN
+F 0 "BT401" H 1168 2146 50  0000 L CNN
 F 1 "Battery_Cell" H 1168 2055 50  0000 L CNN
 F 2 "Battery:BatteryHolder_Keystone_1042_1x18650" V 1050 2110 50  0001 C CNN
@@
 $EndComp
 $Comp
-L Device:Battery_Cell BT2
+L Device:Battery_Cell BT402
 U 1 1 616223C5
 P 1050 2350
-F 0 "BT2" H 1168 2446 50  0000 L CNN
+F 0 "BT402" H 1168 2446 50  0000 L CNN
 F 1 "Battery_Cell" H 1168 2355 50  0000 L CNN
 F 2 "Battery:BatteryHolder_Keystone_1042_1x18650" V 1050 2410 50  0001 C CNN
@@
 Connection ~ 1650 2650
 $Comp
-L power:+BATT #PWR033
+L power:+BATT #PWR0401
 U 1 1 616386ED
 P 1050 1550
-F 0 "#PWR033" H 1050 1400 50  0001 C CNN
+F 0 "#PWR0401" H 1050 1400 50  0001 C CNN
 F 1 "+BATT" H 1065 1723 50  0000 C CNN
 F 2 "" H 1050 1550 50  0001 C CNN
@@
 Connection ~ 2150 4500
 $Comp
-L power:+5V #PWR040
+L power:+5V #PWR0406
 U 1 1 6168DE84
 P 4450 4000
-F 0 "#PWR040" H 4450 3850 50  0001 C CNN
+F 0 "#PWR0406" H 4450 3850 50  0001 C CNN
 F 1 "+5V" V 4450 4200 50  0000 C CNN
 F 2 "" H 4450 4000 50  0001 C CNN
@@
 $EndComp
 $Comp
-L power:GND #PWR039
+L power:GND #PWR0407
 U 1 1 6168E347
 P 4450 4100
-F 0 "#PWR039" H 4450 3850 50  0001 C CNN
+F 0 "#PWR0407" H 4450 3850 50  0001 C CNN
 F 1 "GND" V 4450 3900 50  0000 C CNN
 F 2 "" H 4450 4100 50  0001 C CNN
@@
 $EndComp
 $Comp
-L Connector_Generic:Conn_01x04 J5
+L Connector_Generic:Conn_01x04 J401
 U 1 1 616A0CC6
 P 4650 4100
-F 0 "J5" H 4730 4092 50  0000 L CNN
+F 0 "J401" H 4730 4092 50  0000 L CNN
 F 1 "Conn_01x04" H 4730 4001 50  0000 L CNN
 F 2 "Connector_JST:JST_PH_B4B-PH-K_1x04_P2.00mm_Vertical" H 4650 4100 50  0001 C CNN
@@
 $EndComp
 $Comp
-L power:+BATT #PWR0103
+L power:+BATT #PWR0408
 U 1 1 616AC55C
 P 4450 4200
-F 0 "#PWR0103" H 4450 4050 50  0001 C CNN
+F 0 "#PWR0408" H 4450 4050 50  0001 C CNN
 F 1 "+BATT" V 4450 4450 50  0000 C CNN
 F 2 "" H 4450 4200 50  0001 C CNN
@@
 $EndComp
 $Comp
-L power:GND #PWR0104
+L power:GND #PWR0409
 U 1 1 616AD750
 P 4450 4300
-F 0 "#PWR0104" H 4450 4050 50  0001 C CNN
+F 0 "#PWR0409" H 4450 4050 50  0001 C CNN
 F 1 "GND" V 4450 4100 50  0000 C CNN
 F 2 "" H 4450 4300 50  0001 C CNN

Commit message: Preliminary PCB Production files
Parts:
- C403: LCSC (none) -> C96446; LCSC Part # (none) -> C96446
Changed lines of the file:
@@
 F 2 "Capacitor_SMD:C_0603_1608Metric" H 2588 4200 50  0001 C CNN
 F 3 "~" H 2550 4350 50  0001 C CNN
+F 4 "C96446" H 2550 4350 50  0001 C CNN "LCSC Part #"
+F 5 "C96446" H 2550 4350 50  0001 C CNN "LCSC"
 	1    2550 4350
 	1    0    0    -1

Commit message: Battery board changes
Connections:
- net labels added: CB, FEEDBACK, SWITCH_OUT
Changed lines of the file:
@@
 $Descr A4 11693 8268
 encoding utf-8
-Sheet 4 4
+Sheet 1 1
 Title "Atlas Power Board"
 Date "2021-10-08"
@@
 Text Notes 3900 3450 0    118  ~ 24
 Power Output Connector
+Text Label 6550 2400 0    50   ~ 0
+FEEDBACK
+Text Label 5050 1200 0    50   ~ 0
+SWITCH_OUT
+Text Label 3100 1200 0    50   ~ 0
+CB
 $EndSCHEMATC

Commit message: More changes to battery board, preping for manufacturing
Parts:
- C403: LCSC Part # C96446 -> (none)
- L401: Digikey Part # (none) -> 308-1335-1-ND
- R401: Digikey Part # (none) -> RMCF0805FT3K16CT-ND
- R402, R403: Digikey Part # (none) -> RMCF0805FT1K00CT-ND
- U402: value LM2678T-ADJ_NOPB -> LM2678S-ADJ_NOPB; Digikey Part # (none) -> LM2678S-5.0/NOPB-ND
Changed lines of the file:
@@
 P 4000 1900
 F 0 "U402" H 4000 2367 50  0000 C CNN
-F 1 "LM2678T-ADJ_NOPB" H 4000 2276 50  0000 C CNN
+F 1 "LM2678S-ADJ_NOPB" H 4000 2276 50  0000 C CNN
 F 2 "SamacSys_Parts:TO127P1435X464-8N" H 4000 1900 50  0001 L BNN
 F 3 "" H 4000 1900 50  0001 L BNN
 F 4 "TEXAS INSTRUMENTS" H 4000 1900 50  0001 L BNN "MANUFACTURER"
+F 5 "LM2678S-5.0/NOPB-ND" H 4000 1900 50  0001 C CNN "Digikey Part #"
 	1    4000 1900
 	1    0    0    -1
@@
 F 2 "Resistor_SMD:R_0805_2012Metric" V 7180 1950 50  0001 C CNN
 F 3 "~" H 7250 1950 50  0001 C CNN
+F 4 "RMCF0805FT3K16CT-ND" H 7250 1950 50  0001 C CNN "Digikey Part #"
 	1    7250 1950
 	1    0    0    -1
@@
 F 2 "Resistor_SMD:R_0805_2012Metric" V 7180 2400 50  0001 C CNN
 F 3 "~" H 7250 2400 50  0001 C CNN
+F 4 "RMCF0805FT1K00CT-ND" H 7250 2400 50  0001 C CNN "Digikey Part #"
 	1    7250 2400
 	1    0    0    -1
@@
 F 2 "Inductor_SMD:L_TDK_NLV32_3.2x2.5mm" H 5300 1700 50  0001 C CNN
 F 3 "~" H 5300 1700 50  0001 C CNN
+F 4 "308-1335-1-ND" H 5300 1700 50  0001 C CNN "Digikey Part #"
 	1    5300 1700
 	0    -1   -1   0
@@
 F 2 "Resistor_SMD:R_0805_2012Metric" V 7730 2400 50  0001 C CNN
 F 3 "~" H 7800 2400 50  0001 C CNN
+F 4 "RMCF0805FT1K00CT-ND" H 7800 2400 50  0001 C CNN "Digikey Part #"
 	1    7800 2400
 	1    0    0    -1
@@
 F 2 "Capacitor_SMD:C_0603_1608Metric" H 2588 4200 50  0001 C CNN
 F 3 "~" H 2550 4350 50  0001 C CNN
-F 4 "C96446" H 2550 4350 50  0001 C CNN "LCSC Part #"
+F 4 "" H 2550 4350 50  0001 C CNN "LCSC Part #"
 F 5 "C96446" H 2550 4350 50  0001 C CNN "LCSC"
 	1    2550 4350

Commit message: Battery board sent to fab
Parts:
- C402, C404, C405: Digikey Part # (none) -> 399-11939-1-ND
- D401: Digikey Part # (none) -> 846-RB050LAM-30CT-ND
- D402: Digikey Part # (none) -> 67-1553-1-ND
- L401: footprint Inductor_SMD:L_TDK_NLV32_3.2x2.5mm -> SamacSys_Parts:CDRH127
Changed lines of the file:
@@
 F 2 "Capacitor_SMD:C_0805_2012Metric" H 2488 1950 50  0001 C CNN
 F 3 "~" H 2450 2100 50  0001 C CNN
+F 4 "399-11939-1-ND" H 2450 2100 50  0001 C CNN "Digikey Part #"
 	1    2450 2100
 	1    0    0    -1
@@
 F 2 "Capacitor_SMD:C_0805_2012Metric" H 5988 2000 50  0001 C CNN
 F 3 "~" H 5950 2150 50  0001 C CNN
+F 4 "399-11939-1-ND" H 5950 2150 50  0001 C CNN "Digikey Part #"
 	1    5950 2150
 	1    0    0    -1
@@
 F 2 "Diode_SMD:D_SOD-128" H 5050 2150 50  0001 C CNN
 F 3 "~" H 5050 2150 50  0001 C CNN
+F 4 "846-RB050LAM-30CT-ND" H 5050 2150 50  0001 C CNN "Digikey Part #"
 	1    5050 2150
 	0    1    1    0
@@
 F 0 "L401" V 5490 1700 50  0000 C CNN
 F 1 "22 uH" V 5399 1700 50  0000 C CNN
-F 2 "Inductor_SMD:L_TDK_NLV32_3.2x2.5mm" H 5300 1700 50  0001 C CNN
+F 2 "SamacSys_Parts:CDRH127" H 5300 1700 50  0001 C CNN
 F 3 "~" H 5300 1700 50  0001 C CNN
 F 4 "308-1335-1-ND" H 5300 1700 50  0001 C CNN "Digikey Part #"
@@
 F 2 "Capacitor_SMD:C_0805_2012Metric" H 3888 1050 50  0001 C CNN
 F 3 "~" H 3850 1200 50  0001 C CNN
+F 4 "399-11939-1-ND" H 3850 1200 50  0001 C CNN "Digikey Part #"
 	1    3850 1200
 	0    1    1    0
@@
 F 2 "LED_SMD:LED_0805_2012Metric" H 7800 1950 50  0001 C CNN
 F 3 "~" H 7800 1950 50  0001 C CNN
+F 4 "67-1553-1-ND" H 7800 1950 50  0001 C CNN "Digikey Part #"
 	1    7800 1950
 	0    -1   -1   0
