File: cad/electronics/AtlasPD/5V Buck Converter.sch (KiCad schematic (older format))
At the start: 17 parts, among them J401 Conn_01x04, U401 AMS1117-3.3, U402 LM2678S-ADJ_NOPB

Commit message: 5V Regulator changes
Parts:
- added C1, C2: 10uF, Capacitor_SMD:C_0805_2012Metric, symbol Device:C
- added D1: D_Schottky, Diode_SMD:D_SOD-128, symbol Device:D_Schottky
- added D2: LED, LED_SMD:LED_0805_2012Metric, symbol Device:LED
- added L1: 22 uH, SamacSys_Parts:CDRH127, symbol Device:L
- added R1: 1k, Resistor_SMD:R_0805_2012Metric, symbol Device:R
- added U403: AP1509-50SG-13, symbol SamacSys_Parts:AP1509
Connections:
- wire segments 56 -> 83
Changed lines of the file:
@@
 	7800 2650 7250 2650
 Connection ~ 7250 2650
-Text Notes 2750 1200 2    118  ~ 24
+Text Notes 3200 5900 2    118  ~ 24
 5V Buck Converter
 NoConn ~ 3300 1800
@@
 Text Label 3100 1200 0    50   ~ 0
 CB
+$Comp
+L Device:D_Schottky D1
+U 1 1 61AFE8B4
+P 3900 6950
+F 0 "D1" V 3854 7030 50  0000 L CNN
+F 1 "D_Schottky" V 3945 7030 50  0000 L CNN
+F 2 "Diode_SMD:D_SOD-128" H 3900 6950 50  0001 C CNN
+F 3 "~" H 3900 6950 50  0001 C CNN
+F 4 "846-RB050LAM-30CT-ND" H 3900 6950 50  0001 C CNN "Digikey Part #"
+	1    3900 6950
+	0    1    1    0
+$EndComp
+$Comp
+L Device:L L1
+U 1 1 61B0184A
+P 4350 6600
+F 0 "L1" V 4540 6600 50  0000 C CNN
+F 1 "22 uH" V 4449 6600 50  0000 C CNN
+F 2 "SamacSys_Parts:CDRH127" H 4350 6600 50  0001 C CNN
+F 3 "~" H 4350 6600 50  0001 C CNN
+F 4 "308-1335-1-ND" H 4350 6600 50  0001 C CNN "Digikey Part #"
+	1    4350 6600
+	0    -1   -1   0
+$EndComp
+$Comp
+L Device:C C2
+U 1 1 61B043BD
+P 4850 6900
+F 0 "C2" H 4965 6946 50  0000 L CNN
+F 1 "10uF" H 4965 6855 50  0000 L CNN
+F 2 "Capacitor_SMD:C_0805_2012Metric" H 4888 6750 50  0001 C CNN
+F 3 "~" H 4850 6900 50  0001 C CNN
+F 4 "399-11939-1-ND" H 4850 6900 50  0001 C CNN "Digikey Part #"
+	1    4850 6900
+	1    0    0    -1
+$EndComp
+$Comp
+L Device:C C1
+U 1 1 61B050EC
+P 1600 6900
+F 0 "C1" H 1715 6946 50  0000 L CNN
+F 1 "10uF" H 1715 6855 50  0000 L CNN
+F 2 "Capacitor_SMD:C_0805_2012Metric" H 1638 6750 50  0001 C CNN
+F 3 "~" H 1600 6900 50  0001 C CNN
+F 4 "399-11939-1-ND" H 1600 6900 50  0001 C CNN "Digikey Part #"
+	1    1600 6900
+	1    0    0    -1
+$EndComp
+Wire Wire Line
+	2200 7000 2150 7000
+Wire Wire Line
+	2150 7000 2150 7200
+Wire Wire Line
+	2150 7200 2800 7200
+Wire Wire Line
+	2800 7200 2900 7200
+Connection ~ 2800 7200
+Wire Wire Line
+	3000 7200 2900 7200
+Connection ~ 2900 7200
+Wire Wire Line
+	3100 7200 3000 7200
+Connection ~ 3000 7200
+Wire Wire Line
+	3100 7200 3900 7200
+Wire Wire Line
+	3900 7200 3900 7100
+Connection ~ 3100 7200
+Wire Wire Line
+	3300 6600 3900 6600
+Wire Wire Line
+	3900 6600 3900 6800
+Wire Wire Line
+	3900 6600 4200 6600
+Connection ~ 3900 6600
+Wire Wire Line
+	4500 6600 4850 6600
+Wire Wire Line
+	4850 6600 4850 6750
+Wire Wire Line
+	4850 7050 4850 7200
+Wire Wire Line
+	4850 7200 3900 7200
+Connection ~ 3900 7200
+Wire Wire Line
+	1600 7050 1600 7200
+Wire Wire Line
+	1600 7200 2150 7200
+Connection ~ 2150 7200
+Wire Wire Line
+	1600 6750 1600 6600
+Wire Wire Line
+	1600 6600 2200 6600
+Wire Wire Line
+	2750 6400 2750 6300
+Wire Wire Line
+	2750 6300 4850 6300
+Wire Wire Line
+	4850 6300 4850 6600
+Connection ~ 4850 6600
+$Comp
+L Device:LED D2
+U 1 1 61B2E403
+P 5400 6750
+F 0 "D2" V 5439 6632 50  0000 R CNN
+F 1 "LED" V 5348 6632 50  0000 R CNN
+F 2 "LED_SMD:LED_0805_2012Metric" H 5400 6750 50  0001 C CNN
+F 3 "~" H 5400 6750 50  0001 C CNN
+F 4 "67-1553-1-ND" H 5400 6750 50  0001 C CNN "Digikey Part #"
+	1    5400 6750
+	0    -1   -1   0
+$EndComp
+$Comp
+L Device:R R1
+U 1 1 61B2F8FA
+P 5400 7050
+F 0 "R1" H 5470 7096 50  0000 L CNN
+F 1 "1k" H 5470 7005 50  0000 L CNN
+F 2 "Resistor_SMD:R_0805_2012Metric" V 5330 7050 50  0001 C CNN
+F 3 "~" H 5400 7050 50  0001 C CNN
+F 4 "RMCF0805FT1K00CT-ND" H 5400 7050 50  0001 C CNN "Digikey Part #"
+	1    5400 7050
+	1    0    0    -1
+$EndComp
+Wire Wire Line
+	4850 6600 5400 6600
+Wire Wire Line
+	5400 7200 4850 7200
+Connection ~ 4850 7200
+$Comp
+L SamacSys_Parts:AP1509 U403
+U 1 1 61B17232
+P 2800 6800
+F 0 "U403" H 2300 7150 50  0000 L CNN
+F 1 "AP1509-50SG-13" H 2400 6800 50  0000 L CNN
+F 2 "" H 2570 6870 50  0001 C CNN
+F 3 "" H 2570 6870 50  0001 C CNN
+F 4 "AP1509-50SGDICT-ND - Cut Tape (CT)" H 2800 6800 50  0001 C CNN "Digikey Part #"
+	1    2800 6800
+	1    0    0    -1
+$EndComp
+$Comp
+L power:+BATT #PWR?
+U 1 1 61B3A68E
+P 1600 6500
+F 0 "#PWR?" H 1600 6350 50  0001 C CNN
+F 1 "+BATT" H 1615 6673 50  0000 C CNN
+F 2 "" H 1600 6500 50  0001 C CNN
+F 3 "" H 1600 6500 50  0001 C CNN
+	1    1600 6500
+	1    0    0    -1
+$EndComp
+Connection ~ 1600 6600
+$Comp
+L power:GND #PWR?
+U 1 1 61B3B222
+P 1600 7300
+F 0 "#PWR?" H 1600 7050 50  0001 C CNN
+F 1 "GND" H 1605 7127 50  0000 C CNN
+F 2 "" H 1600 7300 50  0001 C CNN
+F 3 "" H 1600 7300 50  0001 C CNN
+	1    1600 7300
+	1    0    0    -1
+$EndComp
+Connection ~ 1600 7200
+Wire Wire Line
+	1600 7300 1600 7200
+Wire Wire Line
+	1600 6500 1600 6600
+$Comp
+L power:+5V #PWR?
+U 1 1 61B40F7F
+P 5400 6450
+F 0 "#PWR?" H 5400 6300 50  0001 C CNN
+F 1 "+5V" H 5415 6623 50  0000 C CNN
+F 2 "" H 5400 6450 50  0001 C CNN
+F 3 "" H 5400 6450 50  0001 C CNN
+	1    5400 6450
+	1    0    0    -1
+$EndComp
+Wire Wire Line
+	5400 6600 5400 6450
+Connection ~ 5400 6600
 $EndSCHEMATC

Commit message: Battery board Rev 1.5
Parts:
- removed C402, C404, C405: 10uF, Capacitor_SMD:C_0805_2012Metric, symbol Device:C
- removed C406: 1000uF, Capacitor_THT:CP_Radial_D10.0mm_P3.50mm, symbol Device:CP1
- removed D401: D_Schottky, Diode_SMD:D_SOD-128, symbol Device:D_Schottky
- removed D402: LED, LED_SMD:LED_0805_2012Metric, symbol Device:LED
- removed L401: 22 uH, SamacSys_Parts:CDRH127, symbol Device:L
- removed R401: 3.16k, Resistor_SMD:R_0805_2012Metric, symbol Device:R
- removed R402, R403: 1k, Resistor_SMD:R_0805_2012Metric, symbol Device:R
- removed U402: LM2678S-ADJ_NOPB, SamacSys_Parts:TO127P1435X464-8N, symbol LM2678T-ADJ/NOPB:LM2678T-ADJ_NOPB
- added C405: 220uF, Capacitor_THT:CP_Radial_D5.0mm_P2.50mm, symbol Device:CP1
- L401: renamed from L1; value 22 uH -> 39 uH
- U402: renamed from U403; footprint (none) -> Package_SO:SO-8_3.9x4.9mm_P1.27mm
- renumbered C1 to C402, C2 to C404, D1 to D401, D2 to D402, R1 to R401
Connections:
- net labels removed: CB, FEEDBACK, SWITCH_OUT
- wire segments 83 -> 45
- no-connect marks 1 -> 0
Other:
- note added: "Battery Cells"
- moved on the sheet: BT401, BT402, C402, C403, C404, D401, D402, J401, L401, R401, U401, U402
