File: cad/electronics/AtlasPD/5V Buck Converter.sch (KiCad schematic (older format))
At the start: 14 parts, among them J401 Conn_01x04, U401 AMS1117-3.3, U402 AP1509-50SG-13

Commit message: KiCad 6.0 upgrade
Parts:
- C403: LCSC C96446 -> (none)
Changed lines of the file:
@@
 F 3 "~" H 4650 1700 50  0001 C CNN
 F 4 "" H 4650 1700 50  0001 C CNN "LCSC Part #"
-F 5 "C96446" H 4650 1700 50  0001 C CNN "LCSC"
+F 5 "" H 4650 1700 50  0001 C CNN "LCSC"
 	1    4650 1700
 	1    0    0    -1
