File: cad/electronics/AtlasPD/AtlasPD.sch (KiCad schematic (older format))
At the start: 0 parts

Commit message: First Board Layout done
Changed lines of the file:
@@
 F10 "S3" I R 8050 2400 50
 F11 "S4" I R 8050 2500 50
+F12 "EN_MTRS" I R 8050 1100 50
 $EndSheet
 $Sheet
@@
 Text Notes 8100 2900 0    50   ~ 0
 S1/S2: Motor 1\nS3/S4: Motor 2
+Wire Wire Line
+	8050 1100 8550 1100
+Wire Wire Line
+	8550 1100 8550 1000
+Wire Wire Line
+	8550 1000 9100 1000
 $EndSCHEMATC
