File: cad/electronics/AtlasPD/_autosave-AtlasPD.kicad_pcb (KiCad board)
At the start: 4 copper layers, 150.4 x 119.4 mm, 52 parts, among them J1 Conn_01x02_Male, J1 Conn_01x04, J2 Conn_01x02_Male, J2 USB_C_Receptacle_USB2.0, J3 Conn_01x06, J4 Conn_01x06, J5 Conn_01x04, SW1 SW_SPST, U1 CP2104, U2 ATmega328P-AU, U3 74LS08, U4 DRV8837C, U5 DRV8837C, U6 AMS1117-3.3, U7 LM2678T-ADJ_NOPB, Y1 CSTNE16M0V53-R0

Commit message: First Board Layout done
Routing:
- net VCC: vias 19 -> 23
- net GND: vias 57 -> 63
Changed lines of the file:
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@@
   (general
     (thickness 1.6)
-    (drawings 29)
-    (tracks 483)
+    (drawings 28)
+    (tracks 494)
     (zones 0)
     (modules 52)
@@
     (0 F.Cu signal)
     (1 In1.Cu signal hide)
-    (2 In2.Cu signal)
+    (2 In2.Cu signal hide)
     (31 B.Cu signal)
     (32 B.Adhes user)
@@
     (tags capacitor)
     (attr smd)
-    (fp_text reference C5 (at -2.9975 0.0381 135) (layer F.SilkS)
+    (fp_text reference C5 (at -0.176907 -1.454801 135) (layer F.SilkS)
       (effects (font (size 1 1) (thickness 0.15)))
     )
@@
     (descr "JST PH series connector, B4B-PH-K (http://www.jst-mfg.com/product/pdf/eng/ePH.pdf), generated with kicad-footprint-generator")
     (tags "connector JST PH side entry")
-    (fp_text reference J1 (at 3 -2.9 90) (layer F.SilkS)
+    (fp_text reference J1 (at 7.493 -2.8702 180) (layer F.SilkS)
       (effects (font (size 1 1) (thickness 0.15)))
     )
@@
     (tags capacitor)
     (attr smd)
-    (fp_text reference C8 (at -2.4892 0) (layer F.SilkS)
+    (fp_text reference C8 (at -2.4384 -0.0254) (layer F.SilkS)
       (effects (font (size 1 1) (thickness 0.15)))
     )
@@
     (tags "WSON 8 1EP")
     (attr smd)
-    (fp_text reference U4 (at 0.38 -1.9 90) (layer F.SilkS)
+    (fp_text reference U4 (at 0.6858 -2.2796 180) (layer F.SilkS)
       (effects (font (size 1 1) (thickness 0.15)))
     )
@@
     (tags "WSON 8 1EP")
     (attr smd)
-    (fp_text reference U5 (at 0.38 -1.9 90) (layer F.SilkS)
+    (fp_text reference U5 (at 0.5842 -2.2924 180) (layer F.SilkS)
       (effects (font (size 1 1) (thickness 0.15)))
     )
@@
     (tags "SOIC SO")
     (attr smd)
-    (fp_text reference U3 (at 0 -5.28) (layer F.SilkS)
+    (fp_text reference U3 (at -0.0508 5.1308) (layer F.SilkS)
       (effects (font (size 1 1) (thickness 0.15)))
     )
@@
     (descr "JST PH series connector, B6B-PH-K (http://www.jst-mfg.com/product/pdf/eng/ePH.pdf), generated with kicad-footprint-generator")
     (tags "connector JST PH side entry")
-    (fp_text reference J4 (at 5.6896 4.1656) (layer F.SilkS)
+    (fp_text reference J4 (at 11.3218 3.6576) (layer F.SilkS)
       (effects (font (size 1 1) (thickness 0.15)))
     )
@@
     (descr "JST PH series connector, B6B-PH-K (http://www.jst-mfg.com/product/pdf/eng/ePH.pdf), generated with kicad-footprint-generator")
     (tags "connector JST PH side entry")
-    (fp_text reference J3 (at 3.302 4.1656) (layer F.SilkS)
+    (fp_text reference J3 (at 11.302 3.683) (layer F.SilkS)
       (effects (font (size 1 1) (thickness 0.15)))
     )
@@
     (tags "Undefined or Miscellaneous")
     (attr smd)
-    (fp_text reference Y1 (at 0.12237 -2.831709 135) (layer F.SilkS)
+    (fp_text reference Y1 (at 0.266054 -3.262761 135) (layer F.SilkS)
       (effects (font (size 1.27 1.27) (thickness 0.254)))
     )
@@
     (tags "CMS SOT")
     (attr smd)
-    (fp_text reference U6 (at -0.3556 -2.1844) (layer F.SilkS)
+    (fp_text reference U6 (at -5.7404 0.3048) (layer F.SilkS)
       (effects (font (size 1 1) (thickness 0.15)))
     )
@@
     (tags "QFP 0.8")
     (attr smd)
-    (fp_text reference U2 (at -2.191182 -2.478551 45) (layer F.SilkS)
+    (fp_text reference U2 (at -5.172628 -5.24447) (layer F.SilkS)
       (effects (font (size 1 1) (thickness 0.15)))
     )
@@
     (tags resistor)
     (attr smd)
-    (fp_text reference R9 (at -1.5108 1.4224 45) (layer F.SilkS)
+    (fp_text reference R9 (at -0.125724 1.275196 45) (layer F.SilkS)
       (effects (font (size 1 1) (thickness 0.15)))
     )
@@
     (tags resistor)
     (attr smd)
-    (fp_text reference R8 (at 0.0254 1.4605 135) (layer F.SilkS)
+    (fp_text reference R8 (at -0.196382 1.490723 135) (layer F.SilkS)
       (effects (font (size 1 1) (thickness 0.15)))
     )
@@
     (tags resistor)
     (attr smd)
-    (fp_text reference R3 (at -2.2484 -0.4064 180) (layer F.SilkS)
+    (fp_text reference R3 (at -2.1976 -0.381 180) (layer F.SilkS)
       (effects (font (size 1 1) (thickness 0.15)))
     )
@@
     (tags "solder jumper open")
     (attr virtual)
-    (fp_text reference JP1 (at -4.2926 0.1524) (layer F.SilkS)
+    (fp_text reference JP1 (at 0.3048 1.7526) (layer F.SilkS)
       (effects (font (size 1 1) (thickness 0.15)))
     )
@@
     (tags "usb usb-c 2.0 pd")
     (attr smd)
-    (fp_text reference J2 (at -0.0254 0.0254 90) (layer F.SilkS)
+    (fp_text reference J2 (at -5.9436 -0.9652 180) (layer F.SilkS)
       (effects (font (size 1 1) (thickness 0.15)))
     )
@@
     (tags capacitor)
     (attr smd)
-    (fp_text reference C4 (at -0.0889 1.3716 45) (layer F.SilkS)
+    (fp_text reference C4 (at -0.053882 -1.311117 45) (layer F.SilkS)
       (effects (font (size 1 1) (thickness 0.15)))
     )
@@
     (tags capacitor)
     (attr smd)
-    (fp_text reference C3 (at 0.212828 1.490723 45) (layer F.SilkS)
+    (fp_text reference C3 (at -2.550393 0.035921 45) (layer F.SilkS)
       (effects (font (size 1 1) (thickness 0.15)))
     )
@@
     (zone_connect 2)
     (attr smd)
-    (fp_text reference C1 (at -0.0632 1.5748 90) (layer F.SilkS)
+    (fp_text reference C1 (at -0.0124 1.397 90) (layer F.SilkS)
       (effects (font (size 1 1) (thickness 0.15)))
     )
@@
   (gr_line (start 228.0158 31.877) (end 232.3338 31.877) (layer F.SilkS) (width 0.153))
   (gr_line (start 228.0158 26.162) (end 228.0158 31.877) (layer F.SilkS) (width 0.153))
-  (gr_text JLCJLCJLCJLC (at 208.8642 57.0738) (layer F.SilkS)
+  (gr_text JLCJLCJLCJLC (at 205.359 67.0052) (layer F.SilkS)
     (effects (font (size 0.85 0.85) (thickness 0.17)))
   )
   (gr_circle (center 245.4402 45.3898) (end 245.600844 45.3898) (layer F.SilkS) (width 0.3))
-  (gr_text 5V (at 236.7026 42.9006) (layer F.SilkS)
+  (gr_text 5V (at 231.7496 41.5544) (layer F.SilkS)
     (effects (font (size 0.85 0.85) (thickness 0.17)))
   )
-  (gr_text 5V (at 229.997 43.815) (layer F.SilkS)
-    (effects (font (size 0.85 0.85) (thickness 0.17)))
-  )
-  (gr_text 3V3 (at 226.3902 43.815) (layer F.SilkS)
+  (gr_text 3V3 (at 223.9772 41.5544) (layer F.SilkS)
     (effects (font (size 0.85 0.85) (thickness 0.17)))
   )
@@
   (segment (start 258.358008 41.031792) (end 259.334 40.0558) (width 0.5) (layer F.Cu) (net 2))
   (segment (start 258.307208 41.031792) (end 258.358008 41.031792) (width 0.5) (layer F.Cu) (net 2))
+  (via (at 203.5302 35.3314) (size 0.8) (drill 0.4) (layers F.Cu B.Cu) (net 2))
+  (via (at 203.5302 36.6014) (size 0.8) (drill 0.4) (layers F.Cu B.Cu) (net 2))
+  (via (at 203.5556 37.846) (size 0.8) (drill 0.4) (layers F.Cu B.Cu) (net 2))
+  (via (at 202.057 44.069) (size 0.8) (drill 0.4) (layers F.Cu B.Cu) (net 2))
+  (via (at 204.089 44.069) (size 0.8) (drill 0.4) (layers F.Cu B.Cu) (net 2))
+  (via (at 205.9686 44.069) (size 0.8) (drill 0.4) (layers F.Cu B.Cu) (net 2))
   (segment (start 227.1898 39.37) (end 228.7523 39.37) (width 0.5) (layer F.Cu) (net 3))
   (segment (start 121.92 113.3856) (end 120.7008 112.1664) (width 0.897604) (layer F.Cu) (net 4))
@@
   (segment (start 254.849502 44.549325) (end 255.600017 43.79881) (width 0.5) (layer F.Cu) (net 7))
   (segment (start 253.718131 44.549325) (end 254.849502 44.549325) (width 0.5) (layer F.Cu) (net 7))
-  (segment (start 249.023924 49.243532) (end 253.718131 44.549325) (width 0.5) (layer F.Cu) (net 7))
+  (segment (start 249.023924 49.243532) (end 252.067228 46.200228) (width 0.5) (layer F.Cu) (net 7))
   (via (at 246.1006 48.7426) (size 0.8) (drill 0.4) (layers F.Cu B.Cu) (net 7))
   (segment (start 246.1006 49.3776) (end 246.1006 48.7426) (width 0.5) (layer F.Cu) (net 7))
   (segment (start 245.734208 49.743992) (end 246.1006 49.3776) (width 0.5) (layer F.Cu) (net 7))
   (segment (start 245.429408 49.743992) (end 245.734208 49.743992) (width 0.5) (layer F.Cu) (net 7))
+  (segment (start 252.067228 46.200228) (end 253.718131 44.549325) (width 0.5) (layer F.Cu) (net 7))
+  (via (at 252.067228 46.200228) (size 0.8) (drill 0.4) (layers F.Cu B.Cu) (net 7))
+  (via (at 227.9142 46.5582) (size 0.8) (drill 0.4) (layers F.Cu B.Cu) (net 7))
+  (via (at 236.0168 48.5394) (size 0.8) (drill 0.4) (layers F.Cu B.Cu) (net 7))
+  (via (at 236.0168 46.5582) (size 0.8) (drill 0.4) (layers F.Cu B.Cu) (net 7))
   (segment (start 126.111 121.326) (end 126.2888 121.1482) (width 0.897604) (layer F.Cu) (net 8))
   (segment (start 126.111 123.952) (end 126.111 121.326) (width 0.897604) (layer F.Cu) (net 8))
@@
     (polygon
       (pts
-        (xy 214.1982 45.3898) (xy 206.0194 45.3898) (xy 206.0194 39.5478) (xy 214.1982 39.5478)
+        (xy 214.1982 45.3898) (xy 200.9648 45.293007) (xy 201.013275 28.2702) (xy 210.161925 28.2702) (xy 210.1088 39.5478)
+        (xy 214.1982 39.5478)
       )
     )
@@
     (connect_pads yes (clearance 0.2508))
     (min_thickness 0.254)
-    (fill yes (arc_segments 32) (thermal_gap 0.508) (thermal_bridge_width 0.508))
+    (fill yes (arc_segments 32) (thermal_gap 0.508) (thermal_bridge_width 0.508) (smoothing chamfer) (radius 0.5))
     (polygon
       (pts
@@
     (connect_pads yes (clearance 0.2508))
     (min_thickness 0.254)
-    (fill yes (arc_segments 32) (thermal_gap 0.508) (thermal_bridge_width 0.508))
+    (fill yes (arc_segments 32) (thermal_gap 0.508) (thermal_bridge_width 0.508) (smoothing chamfer) (radius 0.5))
     (polygon
       (pts
@@
     (connect_pads yes (clearance 0.2508))
     (min_thickness 0.254)
-    (fill yes (arc_segments 32) (thermal_gap 0.508) (thermal_bridge_width 0.508))
+    (fill yes (arc_segments 32) (thermal_gap 0.508) (thermal_bridge_width 0.508) (smoothing chamfer) (radius 0.5))
     (polygon
       (pts
@@
     (connect_pads yes (clearance 0.2508))
     (min_thickness 0.254)
-    (fill yes (arc_segments 32) (thermal_gap 0.508) (thermal_bridge_width 0.508))
+    (fill yes (arc_segments 32) (thermal_gap 0.508) (thermal_bridge_width 0.508) (smoothing chamfer) (radius 0.5))
     (polygon
       (pts
