File: cad/electronics/AtlasPD/MotorDriver.sch (KiCad schematic (older format))
At the start: 3 parts

Commit message: Added part annotations
Parts:
- gave numbers to parts that had none: 3
Changed lines of the file:
@@
 $EndDescr
 $Comp
-L Connector_Generic:Conn_01x06 J?
+L Connector_Generic:Conn_01x06 J3
 U 1 1 6125E0E9
 P 7900 1950
-F 0 "J?" H 7980 1942 50  0000 L CNN
+F 0 "J3" H 7980 1942 50  0000 L CNN
 F 1 "Conn_01x06" H 7980 1851 50  0000 L CNN
 F 2 "" H 7900 1950 50  0001 C CNN
@@
 -M1
 $Comp
-L power:+5V #PWR?
+L power:+5V #PWR06
 U 1 1 6125FD45
 P 7300 1950
-F 0 "#PWR?" H 7300 1800 50  0001 C CNN
+F 0 "#PWR06" H 7300 1800 50  0001 C CNN
 F 1 "+5V" H 7315 2123 50  0000 C CNN
 F 2 "" H 7300 1950 50  0001 C CNN
@@
 $EndComp
 $Comp
-L power:GND #PWR?
+L power:GND #PWR07
 U 1 1 612604AA
 P 7300 2050
-F 0 "#PWR?" H 7300 1800 50  0001 C CNN
+F 0 "#PWR07" H 7300 1800 50  0001 C CNN
 F 1 "GND" H 7305 1877 50  0000 C CNN
 F 2 "" H 7300 2050 50  0001 C CNN
@@
 S2
 $Comp
-L Connector_Generic:Conn_01x06 J?
+L Connector_Generic:Conn_01x06 J4
 U 1 1 6127A362
 P 7900 2800
-F 0 "J?" H 7980 2792 50  0000 L CNN
+F 0 "J4" H 7980 2792 50  0000 L CNN
 F 1 "Conn_01x06" H 7980 2701 50  0000 L CNN
 F 2 "" H 7900 2800 50  0001 C CNN
@@
 -M2
 $Comp
-L power:+5V #PWR?
+L power:+5V #PWR08
 U 1 1 6127A3C2
 P 7300 2800
-F 0 "#PWR?" H 7300 2650 50  0001 C CNN
+F 0 "#PWR08" H 7300 2650 50  0001 C CNN
 F 1 "+5V" H 7315 2973 50  0000 C CNN
 F 2 "" H 7300 2800 50  0001 C CNN
@@
 $EndComp
 $Comp
-L power:GND #PWR?
+L power:GND #PWR09
 U 1 1 6127A3CC
 P 7300 2900
-F 0 "#PWR?" H 7300 2650 50  0001 C CNN
+F 0 "#PWR09" H 7300 2650 50  0001 C CNN
 F 1 "GND" H 7305 2727 50  0000 C CNN
 F 2 "" H 7300 2900 50  0001 C CNN
@@
 S4
 $Comp
-L Driver_Motor:L298HN U?
+L Driver_Motor:L298HN U3
 U 1 1 6127C4CB
 P 4850 2300
-F 0 "U?" H 4850 3181 50  0000 C CNN
+F 0 "U3" H 4850 3181 50  0000 C CNN
 F 1 "L298HN" H 4850 3090 50  0000 C CNN
 F 2 "Package_TO_SOT_THT:TO-220-15_P2.54x2.54mm_StaggerOdd_Lead4.58mm_Vertical" H 4900 1650 50  0001 L CNN
@@
 	4100 2400 4250 2400
 $Comp
-L power:GND #PWR?
+L power:GND #PWR05
 U 1 1 61280DAC
 P 4850 3150
-F 0 "#PWR?" H 4850 2900 50  0001 C CNN
+F 0 "#PWR05" H 4850 2900 50  0001 C CNN
 F 1 "GND" H 4855 2977 50  0000 C CNN
 F 2 "" H 4850 3150 50  0001 C CNN

Commit message: Layout updates, new PMICs for motors
Parts:
- added U? (x2): DRV8837C, Package_SON:WSON-8-1EP_2x2mm_P0.5mm_EP0.9x1.6mm, symbol Driver_Motor:DRV8837C
Changed lines of the file:
@@
 NoConn ~ 4550 3000
 NoConn ~ 4650 3000
+$Comp
+L Driver_Motor:DRV8837C U?
+U 1 1 61623F54
+P 1700 4100
+F 0 "U?" H 1700 3511 50  0000 C CNN
+F 1 "DRV8837C" H 1700 3420 50  0000 C CNN
+F 2 "Package_SON:WSON-8-1EP_2x2mm_P0.5mm_EP0.9x1.6mm" H 1700 3250 50  0001 C CNN
+F 3 "http://www.ti.com/lit/ds/symlink/drv8837c.pdf" H 1700 4100 50  0001 C CNN
+	1    1700 4100
+	1    0    0    -1
+$EndComp
+$Comp
+L Driver_Motor:DRV8837C U?
+U 1 1 6162467C
+P 3400 4100
+F 0 "U?" H 3400 3511 50  0000 C CNN
+F 1 "DRV8837C" H 3400 3420 50  0000 C CNN
+F 2 "Package_SON:WSON-8-1EP_2x2mm_P0.5mm_EP0.9x1.6mm" H 3400 3250 50  0001 C CNN
+F 3 "http://www.ti.com/lit/ds/symlink/drv8837c.pdf" H 3400 4100 50  0001 C CNN
+	1    3400 4100
+	1    0    0    -1
+$EndComp
 $EndSCHEMATC

Commit message: Added logic gates
Parts:
- removed U3: L298HN, Package_TO_SOT_THT:TO-220-15_P2.54x2.54mm_StaggerOdd_Lead4.58mm_Vertical, symbol Driver_Motor:L298HN
- added U3: 74LS08, Package_SO:SOIC-14_3.9x8.7mm_P1.27mm, symbol 74xx:74LS08
- gave numbers to parts that had none: 2
Connections:
- net labels added: EN, OUT1, OUT2, OUT3, OUT4
- wire segments 23 -> 45
- no-connect marks 2 -> 0
Other:
- moved on the sheet: U6, U7
Changed lines of the file:
@@
 Text HLabel 7600 3100 0    50   Input ~ 0
 S4
+Text HLabel 2400 1400 0    50   Input ~ 0
+IN1
+Text HLabel 2400 2050 0    50   Input ~ 0
+IN2
+Text HLabel 2400 2250 0    50   Input ~ 0
+IN3
+Text HLabel 2400 2850 0    50   Input ~ 0
+IN4
+Text HLabel 2400 1750 0    50   Input ~ 0
+PWM_A
+Text HLabel 2400 2550 0    50   Input ~ 0
+PWM_B
 $Comp
-L Driver_Motor:L298HN U3
-U 1 1 6127C4CB
-P 4850 2300
-F 0 "U3" H 4850 3181 50  0000 C CNN
-F 1 "L298HN" H 4850 3090 50  0000 C CNN
-F 2 "Package_TO_SOT_THT:TO-220-15_P2.54x2.54mm_StaggerOdd_Lead4.58mm_Vertical" H 4900 1650 50  0001 L CNN
-F 3 "http://www.st.com/st-web-ui/static/active/en/resource/technical/document/datasheet/CD00000240.pdf" H 5000 2550 50  0001 C CNN
-	1    4850 2300
+L Driver_Motor:DRV8837C U6
+U 1 1 61623F54
+P 4650 3100
+F 0 "U6" H 4650 2511 50  0000 C CNN
+F 1 "DRV8837C" H 4650 2420 50  0000 C CNN
+F 2 "Package_SON:WSON-8-1EP_2x2mm_P0.5mm_EP0.9x1.6mm" H 4650 2250 50  0001 C CNN
+F 3 "http://www.ti.com/lit/ds/symlink/drv8837c.pdf" H 4650 3100 50  0001 C CNN
+	1    4650 3100
 	1    0    0    -1
 $EndComp
-Text Label 5650 2100 0    50   ~ 0
-+M1
-Text Label 5650 2200 0    50   ~ 0
--M1
-Text Label 5650 2400 0    50   ~ 0
-+M2
-Text Label 5650 2500 0    50   ~ 0
--M2
-Wire Wire Line
-	5450 2100 5650 2100
-Wire Wire Line
-	5450 2200 5650 2200
-Wire Wire Line
-	5450 2400 5650 2400
-Wire Wire Line
-	5450 2500 5650 2500
-Text HLabel 4100 1800 0    50   Input ~ 0
-IN1
-Text HLabel 4100 1900 0    50   Input ~ 0
-IN2
-Text HLabel 4100 2200 0    50   Input ~ 0
-IN3
-Text HLabel 4100 2300 0    50   Input ~ 0
-IN4
-Text HLabel 4100 2000 0    50   Input ~ 0
-PWM_A
-Text HLabel 4100 2400 0    50   Input ~ 0
-PWM_B
-Wire Wire Line
-	4100 1800 4250 1800
-Wire Wire Line
-	4100 1900 4250 1900
-Wire Wire Line
-	4100 2000 4250 2000
-Wire Wire Line
-	4100 2200 4250 2200
-Wire Wire Line
-	4250 2300 4100 2300
-Wire Wire Line
-	4100 2400 4250 2400
 $Comp
-L power:GND #PWR05
-U 1 1 61280DAC
-P 4850 3150
-F 0 "#PWR05" H 4850 2900 50  0001 C CNN
-F 1 "GND" H 4855 2977 50  0000 C CNN
-F 2 "" H 4850 3150 50  0001 C CNN
-F 3 "" H 4850 3150 50  0001 C CNN
-	1    4850 3150
+L Driver_Motor:DRV8837C U7
+U 1 1 6162467C
+P 4650 1400
+F 0 "U7" H 4650 811 50  0000 C CNN
+F 1 "DRV8837C" H 4650 720 50  0000 C CNN
+F 2 "Package_SON:WSON-8-1EP_2x2mm_P0.5mm_EP0.9x1.6mm" H 4650 550 50  0001 C CNN
+F 3 "http://www.ti.com/lit/ds/symlink/drv8837c.pdf" H 4650 1400 50  0001 C CNN
+	1    4650 1400
+	1    0    0    -1
+$EndComp
+$Comp
+L 74xx:74LS08 U3
+U 1 1 61640DB0
+P 3100 1500
+F 0 "U3" H 3100 1825 50  0000 C CNN
+F 1 "74LS08" H 3100 1734 50  0000 C CNN
+F 2 "Package_SO:SOIC-14_3.9x8.7mm_P1.27mm" H 3100 1500 50  0001 C CNN
+F 3 "http://www.ti.com/lit/gpn/sn74LS08" H 3100 1500 50  0001 C CNN
+	1    3100 1500
+	1    0    0    -1
+$EndComp
+$Comp
+L 74xx:74LS08 U3
+U 2 1 616444B9
+P 3100 1950
+F 0 "U3" H 3100 2275 50  0000 C CNN
+F 1 "74LS08" H 3100 2184 50  0000 C CNN
+F 2 "Package_SO:SOIC-14_3.9x8.7mm_P1.27mm" H 3100 1950 50  0001 C CNN
+F 3 "http://www.ti.com/lit/gpn/sn74LS08" H 3100 1950 50  0001 C CNN
+	2    3100 1950
+	1    0    0    -1
+$EndComp
+$Comp
+L 74xx:74LS08 U3
+U 3 1 616454A9
+P 3100 2350
+F 0 "U3" H 3100 2675 50  0000 C CNN
+F 1 "74LS08" H 3100 2584 50  0000 C CNN
+F 2 "Package_SO:SOIC-14_3.9x8.7mm_P1.27mm" H 3100 2350 50  0001 C CNN
+F 3 "http://www.ti.com/lit/gpn/sn74LS08" H 3100 2350 50  0001 C CNN
+	3    3100 2350
+	1    0    0    -1
+$EndComp
+$Comp
+L 74xx:74LS08 U3
+U 4 1 61646528
+P 3100 2750
+F 0 "U3" H 3100 3075 50  0000 C CNN
+F 1 "74LS08" H 3100 2984 50  0000 C CNN
+F 2 "Package_SO:SOIC-14_3.9x8.7mm_P1.27mm" H 3100 2750 50  0001 C CNN
+F 3 "http://www.ti.com/lit/gpn/sn74LS08" H 3100 2750 50  0001 C CNN
+	4    3100 2750
+	1    0    0    -1
+$EndComp
+$Comp
+L 74xx:74LS08 U3
+U 5 1 61647348
+P 1100 2200
+F 0 "U3" H 1330 2246 50  0000 L CNN
+F 1 "74LS08" H 1330 2155 50  0000 L CNN
+F 2 "Package_SO:SOIC-14_3.9x8.7mm_P1.27mm" H 1100 2200 50  0001 C CNN
+F 3 "http://www.ti.com/lit/gpn/sn74LS08" H 1100 2200 50  0001 C CNN
+	5    1100 2200
 	1    0    0    -1
 $EndComp
 Wire Wire Line
-	4850 3150 4850 3000
-NoConn ~ 4550 3000
-NoConn ~ 4650 3000
+	2400 1400 2800 1400
+Wire Wire Line
+	2400 2050 2800 2050
+Wire Wire Line
+	2800 1600 2700 1600
+Wire Wire Line
+	2700 1600 2700 1750
+Wire Wire Line
+	2700 1850 2800 1850
+Wire Wire Line
+	2400 1750 2700 1750
+Connection ~ 2700 1750
+Wire Wire Line
+	2700 1750 2700 1850
+Wire Wire Line
+	2400 2250 2800 2250
+Wire Wire Line
+	2400 2850 2800 2850
+Wire Wire Line
+	2800 2450 2700 2450
+Wire Wire Line
+	2700 2450 2700 2550
+Wire Wire Line
+	2700 2650 2800 2650
+Wire Wire Line
+	2400 2550 2700 2550
+Connection ~ 2700 2550
+Wire Wire Line
+	2700 2550 2700 2650
 $Comp
-L Driver_Motor:DRV8837C U?
-U 1 1 61623F54
-P 1700 4100
-F 0 "U?" H 1700 3511 50  0000 C CNN
-F 1 "DRV8837C" H 1700 3420 50  0000 C CNN
-F 2 "Package_SON:WSON-8-1EP_2x2mm_P0.5mm_EP0.9x1.6mm" H 1700 3250 50  0001 C CNN
-F 3 "http://www.ti.com/lit/ds/symlink/drv8837c.pdf" H 1700 4100 50  0001 C CNN
-	1    1700 4100
+L power:+5V #PWR0105
+U 1 1 61660394
+P 1100 1600
+F 0 "#PWR0105" H 1100 1450 50  0001 C CNN
+F 1 "+5V" H 1115 1773 50  0000 C CNN
+F 2 "" H 1100 1600 50  0001 C CNN
+F 3 "" H 1100 1600 50  0001 C CNN
+	1    1100 1600
 	1    0    0    -1
 $EndComp
 $Comp
-L Driver_Motor:DRV8837C U?
-U 1 1 6162467C
-P 3400 4100
-F 0 "U?" H 3400 3511 50  0000 C CNN
-F 1 "DRV8837C" H 3400 3420 50  0000 C CNN
-F 2 "Package_SON:WSON-8-1EP_2x2mm_P0.5mm_EP0.9x1.6mm" H 3400 3250 50  0001 C CNN
-F 3 "http://www.ti.com/lit/ds/symlink/drv8837c.pdf" H 3400 4100 50  0001 C CNN
-	1    3400 4100
+L power:GND #PWR0106
+U 1 1 61660824
+P 1100 2850
+F 0 "#PWR0106" H 1100 2600 50  0001 C CNN
+F 1 "GND" H 1105 2677 50  0000 C CNN
+F 2 "" H 1100 2850 50  0001 C CNN
+F 3 "" H 1100 2850 50  0001 C CNN
+	1    1100 2850
 	1    0    0    -1
 $EndComp
+Wire Wire Line
+	3400 1500 3750 1500
+Wire Wire Line
+	3750 1500 3750 1400
+Wire Wire Line
+	3750 1400 4250 1400
+Wire Wire Line
+	3400 1950 3900 1950
+Wire Wire Line
+	3900 1950 3900 1500
+Wire Wire Line
+	3900 1500 4250 1500
+Wire Wire Line
+	3400 2750 3750 2750
+Wire Wire Line
+	3750 2750 3750 3200
+Wire Wire Line
+	3750 3200 4250 3200
+Wire Wire Line
+	3400 2350 3900 2350
+Wire Wire Line
+	3900 2350 3900 3100
+Wire Wire Line
+	3900 3100 4250 3100
+Text HLabel 2400 850  0    50   Input ~ 0
+EN
+Wire Wire Line
+	2400 850  4050 850
+Wire Wire Line
+	4050 850  4050 1300
+Wire Wire Line
+	4050 1300 4250 1300
+Wire Wire Line
+	4050 1300 4050 3000
+Wire Wire Line
+	4050 3000 4250 3000
+Connection ~ 4050 1300
+Text Label 3450 1500 0    50   ~ 0
+OUT1
+Text Label 3450 1950 0    50   ~ 0
+OUT2
+Text Label 3450 2350 0    50   ~ 0
+OUT3
+Text Label 3450 2750 0    50   ~ 0
+OUT4
+Wire Wire Line
+	1100 1600 1100 1700
+Wire Wire Line
+	1100 2700 1100 2850
 $EndSCHEMATC

Commit message: Project Restructuring for ease of design and other stuff
Parts:
- J3, J4: footprint (none) -> Connector_JST:JST_PH_B6B-PH-K_1x06_P2.00mm_Vertical
Connections:
- net +M1: now also U7.2 (OUT1)
- net +M2: now also U6.2 (OUT1)
- net -M1: now also U7.3 (OUT2)
- net -M2: now also U6.3 (OUT2)
- net +BATT: now reaches U6.1 (VM)
- net +BATT: now also U7.1 (VM)
- net VCC: now reaches U6.8 (VCC)
- net VCC: now also U7.8 (VCC)
Changed lines of the file:
@@
 encoding utf-8
 Sheet 3 4
-Title ""
-Date ""
-Rev ""
+Title "Motor Driver Board"
+Date "2021-10-08"
+Rev "0.1"
 Comp ""
 Comment1 ""
@@
 F 0 "J3" H 7980 1942 50  0000 L CNN
 F 1 "Conn_01x06" H 7980 1851 50  0000 L CNN
-F 2 "" H 7900 1950 50  0001 C CNN
+F 2 "Connector_JST:JST_PH_B6B-PH-K_1x06_P2.00mm_Vertical" H 7900 1950 50  0001 C CNN
 F 3 "~" H 7900 1950 50  0001 C CNN
 	1    7900 1950
@@
 F 0 "J4" H 7980 2792 50  0000 L CNN
 F 1 "Conn_01x06" H 7980 2701 50  0000 L CNN
-F 2 "" H 7900 2800 50  0001 C CNN
+F 2 "Connector_JST:JST_PH_B6B-PH-K_1x06_P2.00mm_Vertical" H 7900 2800 50  0001 C CNN
 F 3 "~" H 7900 2800 50  0001 C CNN
 	1    7900 2800
@@
 Wire Wire Line
 	1100 2700 1100 2850
+Text Label 5200 1100 0    50   ~ 0
++M1
+Text Label 5200 1700 0    50   ~ 0
+-M1
+Text Label 5200 2800 0    50   ~ 0
++M2
+Text Label 5200 3400 0    50   ~ 0
+-M2
+Wire Wire Line
+	5050 1100 5200 1100
+Wire Wire Line
+	5050 1700 5200 1700
+Wire Wire Line
+	5050 2800 5200 2800
+Wire Wire Line
+	5050 3400 5200 3400
+$Comp
+L power:VCC #PWR?
+U 1 1 6163AB7D
+P 4000 700
+F 0 "#PWR?" H 4000 550 50  0001 C CNN
+F 1 "VCC" H 4015 873 50  0000 C CNN
+F 2 "" H 4000 700 50  0001 C CNN
+F 3 "" H 4000 700 50  0001 C CNN
+	1    4000 700
+	1    0    0    -1
+$EndComp
+$Comp
+L power:+BATT #PWR?
+U 1 1 6163C3B1
+P 4250 700
+F 0 "#PWR?" H 4250 550 50  0001 C CNN
+F 1 "+BATT" H 4265 873 50  0000 C CNN
+F 2 "" H 4250 700 50  0001 C CNN
+F 3 "" H 4250 700 50  0001 C CNN
+	1    4250 700
+	1    0    0    -1
+$EndComp
+Wire Wire Line
+	4250 700  4250 750
+Wire Wire Line
+	4250 750  4650 750
+Wire Wire Line
+	4650 750  4650 900
+Wire Wire Line
+	4000 700  4000 800
+Wire Wire Line
+	4000 800  4100 800
+Wire Wire Line
+	4550 800  4550 900
+Wire Wire Line
+	4100 800  4100 2500
+Wire Wire Line
+	4100 2500 4550 2500
+Wire Wire Line
+	4550 2500 4550 2600
+Connection ~ 4100 800
+Wire Wire Line
+	4100 800  4550 800
+Wire Wire Line
+	4250 750  4200 750
+Wire Wire Line
+	4200 750  4200 2400
+Wire Wire Line
+	4200 2400 4650 2400
+Wire Wire Line
+	4650 2400 4650 2600
+Connection ~ 4250 750
 $EndSCHEMATC

Commit message: Found a bug, squashed it
Connections:
- net +5V: no longer U3.14 (VCC)
- net VCC: now also U3.14 (VCC)
Changed lines of the file:
@@
 	2700 2550 2700 2650
-$Comp
-L power:+5V #PWR0105
-U 1 1 61660394
-P 1100 1600
-F 0 "#PWR0105" H 1100 1450 50  0001 C CNN
-F 1 "+5V" H 1115 1773 50  0000 C CNN
-F 2 "" H 1100 1600 50  0001 C CNN
-F 3 "" H 1100 1600 50  0001 C CNN
-	1    1100 1600
-	1    0    0    -1
-$EndComp
 $Comp
 L power:GND #PWR0106
@@
 	5050 3400 5200 3400
 $Comp
-L power:VCC #PWR?
+L power:VCC #PWR0107
 U 1 1 6163AB7D
 P 4000 700
-F 0 "#PWR?" H 4000 550 50  0001 C CNN
+F 0 "#PWR0107" H 4000 550 50  0001 C CNN
 F 1 "VCC" H 4015 873 50  0000 C CNN
 F 2 "" H 4000 700 50  0001 C CNN
@@
 $EndComp
 $Comp
-L power:+BATT #PWR?
+L power:+BATT #PWR0108
 U 1 1 6163C3B1
 P 4250 700
-F 0 "#PWR?" H 4250 550 50  0001 C CNN
+F 0 "#PWR0108" H 4250 550 50  0001 C CNN
 F 1 "+BATT" H 4265 873 50  0000 C CNN
 F 2 "" H 4250 700 50  0001 C CNN
@@
 	4650 2400 4650 2600
 Connection ~ 4250 750
+$Comp
+L power:VCC #PWR0105
+U 1 1 61698F37
+P 1100 1600
+F 0 "#PWR0105" H 1100 1450 50  0001 C CNN
+F 1 "VCC" H 1115 1773 50  0000 C CNN
+F 2 "" H 1100 1600 50  0001 C CNN
+F 3 "" H 1100 1600 50  0001 C CNN
+	1    1100 1600
+	1    0    0    -1
+$EndComp
 $EndSCHEMATC

Commit message: First Board Layout done
Parts:
- renumbered U7 to U4, U6 to U5
Connections:
- net +M1: now also J3.2 (Pin_2); no longer J3.1 (Pin_1)
- net +M2: now also J4.2 (Pin_2); no longer J4.1 (Pin_1)
- net -M1: now also J3.1 (Pin_1); no longer J3.2 (Pin_2)
- net -M2: now also J4.1 (Pin_1); no longer J4.2 (Pin_2)
- net GND: now also U4.4 (GND), U4.9 (GND), U5.4 (GND), U5.9 (GND)
- net IN1: now also U3.5; no longer U3.1
- net IN2: now also U3.1; no longer U3.5
Changed lines of the file:
@@
 	1    0    0    -1
 $EndComp
+Text Label 7600 1850 2    50   ~ 0
++M1
 Text Label 7600 1750 2    50   ~ 0
-+M1
-Text Label 7600 1850 2    50   ~ 0
 -M1
 $Comp
-L power:+5V #PWR06
+L power:+5V #PWR029
 U 1 1 6125FD45
 P 7300 1950
-F 0 "#PWR06" H 7300 1800 50  0001 C CNN
+F 0 "#PWR029" H 7300 1800 50  0001 C CNN
 F 1 "+5V" H 7315 2123 50  0000 C CNN
 F 2 "" H 7300 1950 50  0001 C CNN
@@
 $EndComp
 $Comp
-L power:GND #PWR07
+L power:GND #PWR030
 U 1 1 612604AA
 P 7300 2050
-F 0 "#PWR07" H 7300 1800 50  0001 C CNN
+F 0 "#PWR030" H 7300 1800 50  0001 C CNN
 F 1 "GND" H 7305 1877 50  0000 C CNN
 F 2 "" H 7300 2050 50  0001 C CNN
@@
 	1    0    0    -1
 $EndComp
+Text Label 7600 2700 2    50   ~ 0
++M2
 Text Label 7600 2600 2    50   ~ 0
-+M2
-Text Label 7600 2700 2    50   ~ 0
 -M2
 $Comp
-L power:+5V #PWR08
+L power:+5V #PWR031
 U 1 1 6127A3C2
 P 7300 2800
-F 0 "#PWR08" H 7300 2650 50  0001 C CNN
+F 0 "#PWR031" H 7300 2650 50  0001 C CNN
 F 1 "+5V" H 7315 2973 50  0000 C CNN
 F 2 "" H 7300 2800 50  0001 C CNN
@@
 $EndComp
 $Comp
-L power:GND #PWR09
+L power:GND #PWR032
 U 1 1 6127A3CC
 P 7300 2900
-F 0 "#PWR09" H 7300 2650 50  0001 C CNN
+F 0 "#PWR032" H 7300 2650 50  0001 C CNN
 F 1 "GND" H 7305 2727 50  0000 C CNN
 F 2 "" H 7300 2900 50  0001 C CNN
@@
 Text HLabel 7600 3100 0    50   Input ~ 0
 S4
+Text HLabel 2400 2050 0    50   Input ~ 0
+IN1
 Text HLabel 2400 1400 0    50   Input ~ 0
-IN1
-Text HLabel 2400 2050 0    50   Input ~ 0
 IN2
 Text HLabel 2400 2250 0    50   Input ~ 0
@@
 PWM_B
 $Comp
-L Driver_Motor:DRV8837C U6
+L Driver_Motor:DRV8837C U5
 U 1 1 61623F54
 P 4650 3100
-F 0 "U6" H 4650 2511 50  0000 C CNN
-F 1 "DRV8837C" H 4650 2420 50  0000 C CNN
+F 0 "U5" H 4900 2650 50  0000 C CNN
+F 1 "DRV8837C" H 4900 2550 50  0000 C CNN
 F 2 "Package_SON:WSON-8-1EP_2x2mm_P0.5mm_EP0.9x1.6mm" H 4650 2250 50  0001 C CNN
 F 3 "http://www.ti.com/lit/ds/symlink/drv8837c.pdf" H 4650 3100 50  0001 C CNN
@@
 $EndComp
 $Comp
-L Driver_Motor:DRV8837C U7
+L Driver_Motor:DRV8837C U4
 U 1 1 6162467C
 P 4650 1400
-F 0 "U7" H 4650 811 50  0000 C CNN
-F 1 "DRV8837C" H 4650 720 50  0000 C CNN
+F 0 "U4" H 4900 950 50  0000 C CNN
+F 1 "DRV8837C" H 4900 850 50  0000 C CNN
 F 2 "Package_SON:WSON-8-1EP_2x2mm_P0.5mm_EP0.9x1.6mm" H 4650 550 50  0001 C CNN
 F 3 "http://www.ti.com/lit/ds/symlink/drv8837c.pdf" H 4650 1400 50  0001 C CNN
@@
 	2700 2550 2700 2650
 $Comp
-L power:GND #PWR0106
+L power:GND #PWR024
 U 1 1 61660824
 P 1100 2850
-F 0 "#PWR0106" H 1100 2600 50  0001 C CNN
+F 0 "#PWR024" H 1100 2600 50  0001 C CNN
 F 1 "GND" H 1105 2677 50  0000 C CNN
 F 2 "" H 1100 2850 50  0001 C CNN
@@
 	5050 3400 5200 3400
 $Comp
-L power:VCC #PWR0107
+L power:VCC #PWR025
 U 1 1 6163AB7D
 P 4000 700
-F 0 "#PWR0107" H 4000 550 50  0001 C CNN
+F 0 "#PWR025" H 4000 550 50  0001 C CNN
 F 1 "VCC" H 4015 873 50  0000 C CNN
 F 2 "" H 4000 700 50  0001 C CNN
@@
 $EndComp
 $Comp
-L power:+BATT #PWR0108
+L power:+BATT #PWR026
 U 1 1 6163C3B1
 P 4250 700
-F 0 "#PWR0108" H 4250 550 50  0001 C CNN
+F 0 "#PWR026" H 4250 550 50  0001 C CNN
 F 1 "+BATT" H 4265 873 50  0000 C CNN
 F 2 "" H 4250 700 50  0001 C CNN
@@
 Connection ~ 4250 750
 $Comp
-L power:VCC #PWR0105
+L power:VCC #PWR023
 U 1 1 61698F37
 P 1100 1600
-F 0 "#PWR0105" H 1100 1450 50  0001 C CNN
+F 0 "#PWR023" H 1100 1450 50  0001 C CNN
 F 1 "VCC" H 1115 1773 50  0000 C CNN
 F 2 "" H 1100 1600 50  0001 C CNN
@@
 	1    0    0    -1
 $EndComp
+$Comp
+L power:GND #PWR028
+U 1 1 616C1A28
+P 4650 3600
+F 0 "#PWR028" H 4650 3350 50  0001 C CNN
+F 1 "GND" H 4655 3427 50  0000 C CNN
+F 2 "" H 4650 3600 50  0001 C CNN
+F 3 "" H 4650 3600 50  0001 C CNN
+	1    4650 3600
+	1    0    0    -1
+$EndComp
+$Comp
+L power:GND #PWR027
+U 1 1 616C2741
+P 4650 1900
+F 0 "#PWR027" H 4650 1650 50  0001 C CNN
+F 1 "GND" H 4655 1727 50  0000 C CNN
+F 2 "" H 4650 1900 50  0001 C CNN
+F 3 "" H 4650 1900 50  0001 C CNN
+	1    4650 1900
+	1    0    0    -1
+$EndComp
