File: cad/electronics/AtlasPD/MotorDriver.sch (KiCad schematic (older format))
At the start: 5 parts, among them J3 Conn_01x06, J4 Conn_01x06, U3 74LS08, U4 DRV8837C, U5 DRV8837C

Commit message: Layout updates
Parts:
- renumbered J3 to J301, J4 to J302, U3 to U301, U4 to U302, U5 to U303
Changed lines of the file:
@@
 $EndDescr
 $Comp
-L Connector_Generic:Conn_01x06 J3
+L Connector_Generic:Conn_01x06 J301
 U 1 1 6125E0E9
 P 7900 1950
-F 0 "J3" H 7980 1942 50  0000 L CNN
+F 0 "J301" H 7980 1942 50  0000 L CNN
 F 1 "Conn_01x06" H 7980 1851 50  0000 L CNN
 F 2 "Connector_JST:JST_PH_B6B-PH-K_1x06_P2.00mm_Vertical" H 7900 1950 50  0001 C CNN
@@
 -M1
 $Comp
-L power:+5V #PWR029
+L power:+5V #PWR0307
 U 1 1 6125FD45
 P 7300 1950
-F 0 "#PWR029" H 7300 1800 50  0001 C CNN
+F 0 "#PWR0307" H 7300 1800 50  0001 C CNN
 F 1 "+5V" H 7315 2123 50  0000 C CNN
 F 2 "" H 7300 1950 50  0001 C CNN
@@
 $EndComp
 $Comp
-L power:GND #PWR030
+L power:GND #PWR0308
 U 1 1 612604AA
 P 7300 2050
-F 0 "#PWR030" H 7300 1800 50  0001 C CNN
+F 0 "#PWR0308" H 7300 1800 50  0001 C CNN
 F 1 "GND" H 7305 1877 50  0000 C CNN
 F 2 "" H 7300 2050 50  0001 C CNN
@@
 S2
 $Comp
-L Connector_Generic:Conn_01x06 J4
+L Connector_Generic:Conn_01x06 J302
 U 1 1 6127A362
 P 7900 2800
-F 0 "J4" H 7980 2792 50  0000 L CNN
+F 0 "J302" H 7980 2792 50  0000 L CNN
 F 1 "Conn_01x06" H 7980 2701 50  0000 L CNN
 F 2 "Connector_JST:JST_PH_B6B-PH-K_1x06_P2.00mm_Vertical" H 7900 2800 50  0001 C CNN
@@
 -M2
 $Comp
-L power:+5V #PWR031
+L power:+5V #PWR0309
 U 1 1 6127A3C2
 P 7300 2800
-F 0 "#PWR031" H 7300 2650 50  0001 C CNN
+F 0 "#PWR0309" H 7300 2650 50  0001 C CNN
 F 1 "+5V" H 7315 2973 50  0000 C CNN
 F 2 "" H 7300 2800 50  0001 C CNN
@@
 $EndComp
 $Comp
-L power:GND #PWR032
+L power:GND #PWR0310
 U 1 1 6127A3CC
 P 7300 2900
-F 0 "#PWR032" H 7300 2650 50  0001 C CNN
+F 0 "#PWR0310" H 7300 2650 50  0001 C CNN
 F 1 "GND" H 7305 2727 50  0000 C CNN
 F 2 "" H 7300 2900 50  0001 C CNN
@@
 PWM_B
 $Comp
-L Driver_Motor:DRV8837C U5
+L Driver_Motor:DRV8837C U303
 U 1 1 61623F54
 P 4650 3100
-F 0 "U5" H 4900 2650 50  0000 C CNN
+F 0 "U303" H 4900 2650 50  0000 C CNN
 F 1 "DRV8837C" H 4900 2550 50  0000 C CNN
 F 2 "Package_SON:WSON-8-1EP_2x2mm_P0.5mm_EP0.9x1.6mm" H 4650 2250 50  0001 C CNN
@@
 $EndComp
 $Comp
-L Driver_Motor:DRV8837C U4
+L Driver_Motor:DRV8837C U302
 U 1 1 6162467C
 P 4650 1400
-F 0 "U4" H 4900 950 50  0000 C CNN
+F 0 "U302" H 4900 950 50  0000 C CNN
 F 1 "DRV8837C" H 4900 850 50  0000 C CNN
 F 2 "Package_SON:WSON-8-1EP_2x2mm_P0.5mm_EP0.9x1.6mm" H 4650 550 50  0001 C CNN
@@
 $EndComp
 $Comp
-L 74xx:74LS08 U3
+L 74xx:74LS08 U301
 U 1 1 61640DB0
 P 3100 1500
-F 0 "U3" H 3100 1825 50  0000 C CNN
+F 0 "U301" H 3100 1825 50  0000 C CNN
 F 1 "74LS08" H 3100 1734 50  0000 C CNN
 F 2 "Package_SO:SOIC-14_3.9x8.7mm_P1.27mm" H 3100 1500 50  0001 C CNN
@@
 $EndComp
 $Comp
-L 74xx:74LS08 U3
+L 74xx:74LS08 U301
 U 2 1 616444B9
 P 3100 1950
-F 0 "U3" H 3100 2275 50  0000 C CNN
+F 0 "U301" H 3100 2275 50  0000 C CNN
 F 1 "74LS08" H 3100 2184 50  0000 C CNN
 F 2 "Package_SO:SOIC-14_3.9x8.7mm_P1.27mm" H 3100 1950 50  0001 C CNN
@@
 $EndComp
 $Comp
-L 74xx:74LS08 U3
+L 74xx:74LS08 U301
 U 3 1 616454A9
 P 3100 2350
-F 0 "U3" H 3100 2675 50  0000 C CNN
+F 0 "U301" H 3100 2675 50  0000 C CNN
 F 1 "74LS08" H 3100 2584 50  0000 C CNN
 F 2 "Package_SO:SOIC-14_3.9x8.7mm_P1.27mm" H 3100 2350 50  0001 C CNN
@@
 $EndComp
 $Comp
-L 74xx:74LS08 U3
+L 74xx:74LS08 U301
 U 4 1 61646528
 P 3100 2750
-F 0 "U3" H 3100 3075 50  0000 C CNN
+F 0 "U301" H 3100 3075 50  0000 C CNN
 F 1 "74LS08" H 3100 2984 50  0000 C CNN
 F 2 "Package_SO:SOIC-14_3.9x8.7mm_P1.27mm" H 3100 2750 50  0001 C CNN
@@
 $EndComp
 $Comp
-L 74xx:74LS08 U3
+L 74xx:74LS08 U301
 U 5 1 61647348
 P 1100 2200
-F 0 "U3" H 1330 2246 50  0000 L CNN
+F 0 "U301" H 1330 2246 50  0000 L CNN
 F 1 "74LS08" H 1330 2155 50  0000 L CNN
 F 2 "Package_SO:SOIC-14_3.9x8.7mm_P1.27mm" H 1100 2200 50  0001 C CNN
@@
 	2700 2550 2700 2650
 $Comp
-L power:GND #PWR024
+L power:GND #PWR0302
 U 1 1 61660824
 P 1100 2850
-F 0 "#PWR024" H 1100 2600 50  0001 C CNN
+F 0 "#PWR0302" H 1100 2600 50  0001 C CNN
 F 1 "GND" H 1105 2677 50  0000 C CNN
 F 2 "" H 1100 2850 50  0001 C CNN
@@
 	5050 3400 5200 3400
 $Comp
-L power:VCC #PWR025
+L power:VCC #PWR0303
 U 1 1 6163AB7D
 P 4000 700
-F 0 "#PWR025" H 4000 550 50  0001 C CNN
+F 0 "#PWR0303" H 4000 550 50  0001 C CNN
 F 1 "VCC" H 4015 873 50  0000 C CNN
 F 2 "" H 4000 700 50  0001 C CNN
@@
 $EndComp
 $Comp
-L power:+BATT #PWR026
+L power:+BATT #PWR0304
 U 1 1 6163C3B1
 P 4250 700
-F 0 "#PWR026" H 4250 550 50  0001 C CNN
+F 0 "#PWR0304" H 4250 550 50  0001 C CNN
 F 1 "+BATT" H 4265 873 50  0000 C CNN
 F 2 "" H 4250 700 50  0001 C CNN
@@
 Connection ~ 4250 750
 $Comp
-L power:VCC #PWR023
+L power:VCC #PWR0301
 U 1 1 61698F37
 P 1100 1600
-F 0 "#PWR023" H 1100 1450 50  0001 C CNN
+F 0 "#PWR0301" H 1100 1450 50  0001 C CNN
 F 1 "VCC" H 1115 1773 50  0000 C CNN
 F 2 "" H 1100 1600 50  0001 C CNN
@@
 $EndComp
 $Comp
-L power:GND #PWR028
+L power:GND #PWR0306
 U 1 1 616C1A28
 P 4650 3600
-F 0 "#PWR028" H 4650 3350 50  0001 C CNN
+F 0 "#PWR0306" H 4650 3350 50  0001 C CNN
 F 1 "GND" H 4655 3427 50  0000 C CNN
 F 2 "" H 4650 3600 50  0001 C CNN
@@
 $EndComp
 $Comp
-L power:GND #PWR027
+L power:GND #PWR0305
 U 1 1 616C2741
 P 4650 1900
-F 0 "#PWR027" H 4650 1650 50  0001 C CNN
+F 0 "#PWR0305" H 4650 1650 50  0001 C CNN
 F 1 "GND" H 4655 1727 50  0000 C CNN
 F 2 "" H 4650 1900 50  0001 C CNN
