File: cad/electronics/AtlasPD/MotorDriver.sch (KiCad schematic (older format))
At the start: 5 parts, among them J301 Conn_01x06, J302 Conn_01x06, U301 74LS08, U302 DRV8837C, U303 DRV8837C

Commit message: Preliminary PCB Production files
Parts:
- U301: LCSC (none) -> C5593; LCSC Part # (none) -> C5593
- U302, U303: LCSC (none) -> C191000; LCSC Part # (none) -> C191000
Changed lines of the file:
@@
 F 2 "Package_SON:WSON-8-1EP_2x2mm_P0.5mm_EP0.9x1.6mm" H 4650 2250 50  0001 C CNN
 F 3 "http://www.ti.com/lit/ds/symlink/drv8837c.pdf" H 4650 3100 50  0001 C CNN
+F 4 "C191000" H 4650 3100 50  0001 C CNN "LCSC Part #"
+F 5 "C191000" H 4650 3100 50  0001 C CNN "LCSC"
 	1    4650 3100
 	1    0    0    -1
@@
 F 2 "Package_SON:WSON-8-1EP_2x2mm_P0.5mm_EP0.9x1.6mm" H 4650 550 50  0001 C CNN
 F 3 "http://www.ti.com/lit/ds/symlink/drv8837c.pdf" H 4650 1400 50  0001 C CNN
+F 4 "C191000" H 4650 1400 50  0001 C CNN "LCSC Part #"
+F 5 "C191000" H 4650 1400 50  0001 C CNN "LCSC"
 	1    4650 1400
 	1    0    0    -1
@@
 F 2 "Package_SO:SOIC-14_3.9x8.7mm_P1.27mm" H 3100 1500 50  0001 C CNN
 F 3 "http://www.ti.com/lit/gpn/sn74LS08" H 3100 1500 50  0001 C CNN
+F 4 "C5593" H 3100 1500 50  0001 C CNN "LCSC Part #"
+F 5 "C5593" H 3100 1500 50  0001 C CNN "LCSC"
 	1    3100 1500
 	1    0    0    -1
@@
 F 2 "Package_SO:SOIC-14_3.9x8.7mm_P1.27mm" H 3100 1950 50  0001 C CNN
 F 3 "http://www.ti.com/lit/gpn/sn74LS08" H 3100 1950 50  0001 C CNN
+F 4 "C5593" H 3100 1950 50  0001 C CNN "LCSC Part #"
+F 5 "C5593" H 3100 1950 50  0001 C CNN "LCSC"
 	2    3100 1950
 	1    0    0    -1
@@
 F 2 "Package_SO:SOIC-14_3.9x8.7mm_P1.27mm" H 3100 2350 50  0001 C CNN
 F 3 "http://www.ti.com/lit/gpn/sn74LS08" H 3100 2350 50  0001 C CNN
+F 4 "C5593" H 3100 2350 50  0001 C CNN "LCSC Part #"
+F 5 "C5593" H 3100 2350 50  0001 C CNN "LCSC"
 	3    3100 2350
 	1    0    0    -1
@@
 F 2 "Package_SO:SOIC-14_3.9x8.7mm_P1.27mm" H 3100 2750 50  0001 C CNN
 F 3 "http://www.ti.com/lit/gpn/sn74LS08" H 3100 2750 50  0001 C CNN
+F 4 "C5593" H 3100 2750 50  0001 C CNN "LCSC Part #"
+F 5 "C5593" H 3100 2750 50  0001 C CNN "LCSC"
 	4    3100 2750
 	1    0    0    -1
@@
 F 2 "Package_SO:SOIC-14_3.9x8.7mm_P1.27mm" H 1100 2200 50  0001 C CNN
 F 3 "http://www.ti.com/lit/gpn/sn74LS08" H 1100 2200 50  0001 C CNN
+F 4 "C5593" H 1100 2200 50  0001 C CNN "LCSC Part #"
+F 5 "C5593" H 1100 2200 50  0001 C CNN "LCSC"
 	5    1100 2200
 	1    0    0    -1
