File: cad/electronics/AtlasPD/5V Buck Converter.kicad_sch (KiCad schematic)
At the start: 31 parts, among them J401 Conn_01x04, Q401 Q_Dual_NMOS_S1G1S2G2D2D2D1D1, U401 AP1509-50SG-13, U402 DS2777, U403 AMS1117-3.3

Commit message: Fixed schematic issues from KiCAD upgrade, Moved 3.3V LDO to MCU Sheet
Parts:
- removed C408: 10uF, Capacitor_SMD:C_0603_1608Metric, symbol Device:C
- removed U403: AMS1117-3.3, Package_TO_SOT_SMD:SOT-223-3_TabPin2, symbol Regulator_Linear:AMS1117-3.3
- added TP401: SDA, TestPoint:TestPoint_Pad_1.5x1.5mm, symbol Connector:TestPoint_Alt
- added TP402: SCL, TestPoint:TestPoint_Pad_D1.5mm, symbol Connector:TestPoint_Alt
Connections:
- net SCL: now also TP402.1
- net SDA: now also TP401.1
- net BT_VDD: now reaches BT401.1 (+), Q401.5 (D), Q401.6 (D), R402.1, R403.1
Other:
- note removed: "3.3V LDO"

Commit message: Small changes, saving what I have
Connections:
- net SRC: now also Q401.1 (S), Q401.3 (S), R405.1
Changed lines of the file:
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@@
+    (stroke (width 0) (type default) (color 0 0 0 0))
+  )
+  (wire (pts (xy 80.01 41.91) (xy 80.01 44.45))
     (stroke (width 0) (type default) (color 0 0 0 0))
   )
@@
     (effects (font (size 1.27 1.27)) (justify left bottom))
   )
+  (label "SRC" (at 80.01 41.91 0)
+    (effects (font (size 1.27 1.27)) (justify left bottom))
+  )

Commit message: Finished Battery Board V2 PCB Layout
Connections:
- net SRC: no longer Q401.1 (S), Q401.3 (S), R405.1
- new net Q_SRC: Q401.1 (S), Q401.3 (S), R405.1
Changed lines of the file:
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@@
     (effects (font (size 1.27 1.27)) (justify left bottom))
   )
-  (label "SRC" (at 80.01 41.91 0)
+  (label "Q_SRC" (at 80.01 41.91 0)
     (effects (font (size 1.27 1.27)) (justify left bottom))
   )

Commit message: Refined PCB design, want to do final review later on before sending to Fab
Parts:
- R406: value RSNS -> 20m; footprint Resistor_SMD:R_0805_2012Metric -> Resistor_THT:R_Box_L13.0mm_W4.0mm_P9.00mm
Changed lines of the file:
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@@
     (in_bom yes) (on_board yes) (fields_autoplaced)
     (property "Reference" "R406" (id 0) (at 80.01 95.3475 90))
-    (property "Value" "RSNS" (id 1) (at 80.01 98.1226 90))
-    (property "Footprint" "Resistor_SMD:R_0805_2012Metric" (id 2) (at 80.01 102.108 90)
+    (property "Value" "20m" (id 1) (at 80.01 98.1226 90))
+    (property "Footprint" "Resistor_THT:R_Box_L13.0mm_W4.0mm_P9.00mm" (id 2) (at 80.01 102.108 90)
       (effects (font (size 1.27 1.27)) hide)
     )
@@
     )
     (path "/57171975-0c61-495a-bb3b-6550cc5d5f7f"
-      (reference "R406") (unit 1) (value "RSNS") (footprint "Resistor_SMD:R_0805_2012Metric")
+      (reference "R406") (unit 1) (value "20m") (footprint "Resistor_THT:R_Box_L13.0mm_W4.0mm_P9.00mm")
     )
     (path "/96081f1f-4df0-4ce6-bcbe-894b4af08efa"

Commit message: Simplified design layout
Parts:
- R406: footprint Resistor_THT:R_Box_L13.0mm_W4.0mm_P9.00mm -> Resistor_SMD:R_1206_3216Metric_Pad1.30x1.75mm_HandSolder
Changed lines of the file:
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@@
     (property "Reference" "R406" (id 0) (at 80.01 95.3475 90))
     (property "Value" "20m" (id 1) (at 80.01 98.1226 90))
-    (property "Footprint" "Resistor_THT:R_Box_L13.0mm_W4.0mm_P9.00mm" (id 2) (at 80.01 102.108 90)
+    (property "Footprint" "Resistor_SMD:R_1206_3216Metric_Pad1.30x1.75mm_HandSolder" (id 2) (at 80.01 102.108 90)
       (effects (font (size 1.27 1.27)) hide)
     )
@@
     )
     (path "/57171975-0c61-495a-bb3b-6550cc5d5f7f"
-      (reference "R406") (unit 1) (value "20m") (footprint "Resistor_THT:R_Box_L13.0mm_W4.0mm_P9.00mm")
+      (reference "R406") (unit 1) (value "20m") (footprint "Resistor_SMD:R_1206_3216Metric_Pad1.30x1.75mm_HandSolder")
     )
     (path "/96081f1f-4df0-4ce6-bcbe-894b4af08efa"
