File: cad/electronics/AtlasPD/5V Buck Converter.kicad_sch (KiCad schematic)
At the start: 31 parts, among them J401 Conn_01x04, Q401 Q_Dual_NMOS_S1G1S2G2D2D2D1D1, U401 AP1509-50SG-13, U402 DS2777

Commit message: Changing MCU design due to chip shortage affecting current design/plans
Parts:
- R406: value 20m -> RSNS; footprint Resistor_SMD:R_1206_3216Metric_Pad1.30x1.75mm_HandSolder -> Resistor_SMD:R_0805_2012Metric
Changed lines of the file:
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@@
     (in_bom yes) (on_board yes) (fields_autoplaced)
     (property "Reference" "R406" (id 0) (at 80.01 95.3475 90))
-    (property "Value" "20m" (id 1) (at 80.01 98.1226 90))
-    (property "Footprint" "Resistor_SMD:R_1206_3216Metric_Pad1.30x1.75mm_HandSolder" (id 2) (at 80.01 102.108 90)
+    (property "Value" "RSNS" (id 1) (at 80.01 98.1226 90))
+    (property "Footprint" "Resistor_SMD:R_0805_2012Metric" (id 2) (at 80.01 102.108 90)
       (effects (font (size 1.27 1.27)) hide)
     )
