File: cad/electronics/AtlasPD/Microcontroller.kicad_sch (KiCad schematic)
At the start: 34 parts, among them J201 USB_C_Receptacle_USB2.0, J202 Conn_01x04, J203 Conn_02x03_Odd_Even, SW201 SW_SPST, U201 CP2104, U202 ATmega328P-AU, U203 AMS1117-3.3, Y201 16MHz

Commit message: Small changes
Parts:
- C201, C202, C203, C204, C205, C206: footprint Capacitor_SMD:C_0603_1608Metric -> Capacitor_SMD:C_0402_1005Metric
- D201, D202, D203, D204: footprint LED_SMD:LED_0603_1608Metric -> LED_SMD:LED_0402_1005Metric
- R202, R203, R204, R205, R206, R207, R208, R209: footprint Resistor_SMD:R_0603_1608Metric -> Resistor_SMD:R_0402_1005Metric
Changed lines of the file:
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@@
     (property "Reference" "R203" (id 0) (at 55.88 41.91 90))
     (property "Value" "5.11K" (id 1) (at 55.88 40.005 90))
-    (property "Footprint" "Resistor_SMD:R_0603_1608Metric" (id 2) (at 60.96 40.64 0)
+    (property "Footprint" "Resistor_SMD:R_0402_1005Metric" (id 2) (at 60.96 40.64 0)
       (effects (font (size 1.27 1.27)) hide)
     )
@@
     (property "Reference" "R202" (id 0) (at 66.675 36.195 90))
     (property "Value" "5.11K" (id 1) (at 66.675 34.29 90))
-    (property "Footprint" "Resistor_SMD:R_0603_1608Metric" (id 2) (at 66.675 38.1 0)
+    (property "Footprint" "Resistor_SMD:R_0402_1005Metric" (id 2) (at 66.675 38.1 0)
       (effects (font (size 1.27 1.27)) hide)
     )
@@
       (effects (font (size 1.27 1.27)) (justify right))
     )
-    (property "Footprint" "Capacitor_SMD:C_0603_1608Metric" (id 2) (at 107.315 76.2 0)
+    (property "Footprint" "Capacitor_SMD:C_0402_1005Metric" (id 2) (at 107.315 76.2 0)
       (effects (font (size 1.27 1.27)) hide)
     )
@@
       (effects (font (size 1.27 1.27)) (justify right))
     )
-    (property "Footprint" "LED_SMD:LED_0603_1608Metric" (id 2) (at 158.115 57.15 90)
+    (property "Footprint" "LED_SMD:LED_0402_1005Metric" (id 2) (at 158.115 57.15 90)
       (effects (font (size 1.27 1.27)) hide)
     )
@@
       (effects (font (size 1.27 1.27)) (justify right))
     )
-    (property "Footprint" "LED_SMD:LED_0603_1608Metric" (id 2) (at 161.925 59.69 90)
+    (property "Footprint" "LED_SMD:LED_0402_1005Metric" (id 2) (at 161.925 59.69 90)
       (effects (font (size 1.27 1.27)) hide)
     )
@@
     (property "Reference" "R205" (id 0) (at 151.765 64.135 90))
     (property "Value" "1K" (id 1) (at 151.765 62.23 90))
-    (property "Footprint" "Resistor_SMD:R_0603_1608Metric" (id 2) (at 151.765 62.23 0)
+    (property "Footprint" "Resistor_SMD:R_0402_1005Metric" (id 2) (at 151.765 62.23 0)
       (effects (font (size 1.27 1.27)) hide)
     )
@@
     (property "Reference" "R206" (id 0) (at 146.685 57.785 90))
     (property "Value" "1K" (id 1) (at 146.685 59.69 90))
-    (property "Footprint" "Resistor_SMD:R_0603_1608Metric" (id 2) (at 146.685 59.69 0)
+    (property "Footprint" "Resistor_SMD:R_0402_1005Metric" (id 2) (at 146.685 59.69 0)
       (effects (font (size 1.27 1.27)) hide)
     )
@@
       (effects (font (size 1.27 1.27)) (justify right))
     )
-    (property "Footprint" "Capacitor_SMD:C_0603_1608Metric" (id 2) (at 100.965 26.67 0)
+    (property "Footprint" "Capacitor_SMD:C_0402_1005Metric" (id 2) (at 100.965 26.67 0)
       (effects (font (size 1.27 1.27)) hide)
     )
@@
       (effects (font (size 1.27 1.27)) (justify right))
     )
-    (property "Footprint" "Capacitor_SMD:C_0603_1608Metric" (id 2) (at 219.71 27.94 0)
+    (property "Footprint" "Capacitor_SMD:C_0402_1005Metric" (id 2) (at 219.71 27.94 0)
       (effects (font (size 1.27 1.27)) hide)
     )
@@
       (effects (font (size 1.27 1.27)) (justify right))
     )
-    (property "Footprint" "Capacitor_SMD:C_0603_1608Metric" (id 2) (at 227.33 27.94 0)
+    (property "Footprint" "Capacitor_SMD:C_0402_1005Metric" (id 2) (at 227.33 27.94 0)
       (effects (font (size 1.27 1.27)) hide)
     )
@@
       (effects (font (size 1.27 1.27)) (justify right))
     )
-    (property "Footprint" "Resistor_SMD:R_0603_1608Metric" (id 2) (at 245.11 71.12 0)
+    (property "Footprint" "Resistor_SMD:R_0402_1005Metric" (id 2) (at 245.11 71.12 0)
       (effects (font (size 1.27 1.27)) hide)
     )
@@
       (effects (font (size 1.27 1.27)) (justify left))
     )
-    (property "Footprint" "Capacitor_SMD:C_0603_1608Metric" (id 2) (at 250.19 71.12 0)
+    (property "Footprint" "Capacitor_SMD:C_0402_1005Metric" (id 2) (at 250.19 71.12 0)
       (effects (font (size 1.27 1.27)) hide)
     )
@@
     (property "Reference" "R208" (id 0) (at 234.95 80.645 90))
     (property "Value" "1K" (id 1) (at 234.95 82.55 90))
-    (property "Footprint" "Resistor_SMD:R_0603_1608Metric" (id 2) (at 234.95 82.55 0)
+    (property "Footprint" "Resistor_SMD:R_0402_1005Metric" (id 2) (at 234.95 82.55 0)
       (effects (font (size 1.27 1.27)) hide)
     )
@@
       (effects (font (size 1.27 1.27)) (justify right))
     )
-    (property "Footprint" "LED_SMD:LED_0603_1608Metric" (id 2) (at 92.71 110.49 0)
+    (property "Footprint" "LED_SMD:LED_0402_1005Metric" (id 2) (at 92.71 110.49 0)
       (effects (font (size 1.27 1.27)) hide)
     )
@@
       (effects (font (size 1.27 1.27)) (justify right))
     )
-    (property "Footprint" "LED_SMD:LED_0603_1608Metric" (id 2) (at 110.49 110.49 0)
+    (property "Footprint" "LED_SMD:LED_0402_1005Metric" (id 2) (at 110.49 110.49 0)
       (effects (font (size 1.27 1.27)) hide)
     )
@@
       (effects (font (size 1.27 1.27)) (justify left))
     )
-    (property "Footprint" "Resistor_SMD:R_0603_1608Metric" (id 2) (at 90.932 120.65 90)
+    (property "Footprint" "Resistor_SMD:R_0402_1005Metric" (id 2) (at 90.932 120.65 90)
       (effects (font (size 1.27 1.27)) hide)
     )
@@
       (effects (font (size 1.27 1.27)) (justify left))
     )
-    (property "Footprint" "Resistor_SMD:R_0603_1608Metric" (id 2) (at 108.712 120.65 90)
+    (property "Footprint" "Resistor_SMD:R_0402_1005Metric" (id 2) (at 108.712 120.65 90)
       (effects (font (size 1.27 1.27)) hide)
     )
@@
       (effects (font (size 1.27 1.27)) (justify left))
     )
-    (property "Footprint" "Capacitor_SMD:C_0603_1608Metric" (id 2) (at 158.4452 121.92 0)
-      (effects (font (size 1.27 1.27)) hide)
-    )
+    (property "Footprint" "Capacitor_SMD:C_0402_1005Metric" (id 2) (at 158.4452 121.92 0)
+      (effects (font (size 1.27 1.27)) hide)
+    )
