File: cad/electronics/DronePowerDelivery_Project/DronePowerDelivery/DronePowerDelivery.kicad_pcb (KiCad board)
At the start: 2 copper layers, 52.6 x 56.4 mm, 42 parts, among them J1 Conn_01x05_Socket, J2 Conn_01x02_Socket, J3 Conn_01x04_Pin, J4 Conn_01x02_Socket, Q1 Q_NMOS_GDS, Q2 Q_NMOS_GDS, Q3 Q_PMOS_GSD, SW1 SW_Push, U1 BQ76920PW

Commit message: Rev.1 of PCB laid out
Parts:
- TP1, TP2, TP3, TP4, TP5, TP6: footprint TestPoint:TestPoint_Pad_3.0x3.0mm -> TestPoint:TestPoint_Pad_2.0x2.0mm
- moved J3 12.6 mm to (86.0, 84.2)
- moved R12 12.5 mm to (94.0, 97.9)
- moved R6 11.2 mm to (113.3, 95.8)
- moved C7 10.9 mm to (112.5, 93.1)
- moved R7 10.7 mm to (111.3, 95.8)
- moved R11 10.5 mm to (109.3, 95.8)
- moved D1 10.5 mm to (95.2, 95.2)
- moved SW1 9.46 mm to (101.5, 94.8)
- moved R13 9.31 mm to (96.2, 97.9)
- moved Q3 5.58 mm to (101.8, 99.7), turned to 90 degrees
- moved R1 5.07 mm to (112.6, 90.2)
- moved R2 4.81 mm to (112.6, 88.5)
- moved R5 4.69 mm to (112.6, 82.8)
- moved R3 4.67 mm to (112.6, 86.8)
- moved R4 4.66 mm to (112.6, 85.0)
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Routing:
- net /PACK_H: track 5.18 -> 52.9 mm, vias 0 -> 1
- net /ALERT: track 0.00 -> 40.2 mm, vias 0 -> 1
- net /SCL: track 0.00 -> 34.7 mm, vias 0 -> 1
- net /CellMonitor/CHG: track 0.00 -> 26.3 mm, vias 0 -> 2
- net /SDA: track 0.00 -> 25.8 mm
- net /CellMonitor/SRP: track 6.23 -> 29.7 mm, vias 0 -> 2
- net /CellMonitor/SRN: track 4.62 -> 25.9 mm, vias 0 -> 2
- net /CellMonitor/DSG: track 0.00 -> 20.9 mm, vias 0 -> 2
- net Net-(U1-TS1): track 0.00 -> 18.5 mm, vias 0 -> 2
- net /REGOUT: track 4.63 -> 22.1 mm, vias 0 -> 2
- net /PACK_L: track 0.00 -> 14.9 mm
- net /CellMonitor/Q1_SRC: track 0.00 -> 9.59 mm
- net /CellMonitor/CELL1_Low: track 14.2 -> 23.4 mm
- net Net-(R10-Pad1): track 0.00 -> 8.14 mm
- net Net-(D1-A): track 0.00 -> 8.12 mm
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- added copper zone on F.Cu, net /CellMonitor/Q_DRN
- added copper zone on B.Cu, net /PACK_H
- added copper zone on B.Cu, net GNDREF
- added copper zone on F.Cu, net GNDREF
- added copper zone on In1.Cu, net GNDREF
- added copper zone on In2.Cu, net GNDREF
Other:
- copper layers 2 -> 4

Commit message: Finalied Rev1 Layout
Parts:
- added G***: LOGO, LOGO, B.Cu at (105.5, 95.8)
- added REF**: MountingHole_2.2mm_M2_ISO14580, MountingHole:MountingHole_2.2mm_M2_ISO14580, F.Cu at (85.6, 100.0)
- added REF**: MountingHole_2.2mm_M2_ISO14580, MountingHole:MountingHole_2.2mm_M2_ISO14580, F.Cu at (123.2, 99.8)
- added REF**: MountingHole_2.2mm_M2_ISO14580, MountingHole:MountingHole_2.2mm_M2_ISO14580, F.Cu at (123.2, 75.8)
- added REF**: MountingHole_2.2mm_M2_ISO14580, MountingHole:MountingHole_2.2mm_M2_ISO14580, F.Cu at (85.6, 75.8)
- added kibuzzard-64ABA4C5: G***, kibuzzard-64ABA4C5, F.Cu at (116.8, 105.3)
- added kibuzzard-64ABA514: G***, kibuzzard-64ABA514, F.Cu at (93.3, 106.1)
- moved TP3 10.2 mm to (92.0, 80.0)
- moved TP5 5.67 mm to (88.5, 80.0)
- moved TP6 5.29 mm to (95.5, 80.0)
- moved R8 4.72 mm to (114.8, 114.4), turned to -90 degrees
- moved J2 4.60 mm to (122.9, 115.3)
- moved J4 4.60 mm to (87.1, 115.2)
- moved Q2 4.60 mm to (98.8, 113.5)
- moved Q1 4.60 mm to (106.7, 111.8)
- moved TP2 3.13 mm to (114.0, 77.3)
- moved TP4 2.73 mm to (106.5, 77.3)
- moved TP1 2.52 mm to (110.2, 77.3)
- moved C10 1.78 mm to (112.6, 80.2)
Routing:
- net /CellMonitor/DSG: track 20.9 -> 47.2 mm, vias 2 -> 3
- net /PACK_L: track 14.9 -> 36.6 mm, vias 0 -> 1
- net /PACK_H: track 52.9 -> 66.8 mm
- net /CellMonitor/Q1_SRC: track 9.59 -> 22.5 mm, vias 0 -> 2
- net /CellMonitor/IN_PROT: track 4.98 -> 16.6 mm, vias 0 -> 2
- net /SDA: track 25.8 -> 21.4 mm
- net GNDREF: track 22.3 -> 18.6 mm, vias 3 -> 30
- net /SCL: track 34.7 -> 37.5 mm
- net /REGOUT: track 22.1 -> 20.4 mm
- net /ALERT: track 40.2 -> 38.5 mm
- added copper zone on F.Cu, net /CellMonitor/Q1_SRC
Other:
- board size 52.6 x 56.4 mm -> 47.4 x 48 mm
- board text added: "3V3"
- board text added: "ALR"
- board text added: "BatPD Rev. 1 M. Singh Jul. 2023"
- board text added: "GND"
- board text added: "SCL"
- board text added: "SDA"

Commit message: Finished and ordered Rev1 of DronePD PCB
Parts:
- moved G*** 11.3 mm to (105.9, 107.1), turned to 180 degrees
- moved REF** 0.90 mm to (124.1, 99.8)
- moved REF** 0.90 mm to (124.1, 75.8)
Routing:
- net GNDREF: vias 30 -> 33
Other:
- outline, holes or cut-outs redrawn
- board text added: "DronePD Rev.1 M. Singh Jul. 2023"
- board text added: "PACK+"
- board text added: "PACK-"
- board text removed: "BatPD Rev. 1 M. Singh Jul. 2023"
